File: hv_power_supply/power_bank/Antoinette_power_bank/Antoinette_power_bank.sch (KiCad schematic (older format))
At the start: 43 parts, among them J1 CONN_01x02, J2 CONN_01x02, J3 USB_A, Q1 SSM3K333R, U1 USB_MicroB, U2 MCP73871T-2CCI_ML, U3 TPS61090RSAR

Commit message: Antoinette's initial power bank schematic completed
Parts:
- removed J3: USB_A, symbol PowerBankTemplate-rescue:USB_A-Connector
- added J3: USB_A, symbol Connector:USB_A
- renumbered C5 to C3, C3 to C4, C4 to C5, D2 to D1, D1 to D2, R9 to R10, R13 to R11, R14 to R12, R17 to R13, R11 to R14, R12 to R15, R15 to R16, R16 to R17, R7 to R5, R8 to R6, R5 to R7, R6 to R8, R10 to R9, TP2 to TP1, TP5 to TP2, TP1 to TP5
Other:
- note removed: "+5V"
- note removed: "Battery+"
- note removed: "MCP"
- note removed: "Micro USB"
- note removed: "Power Flow"
- note removed: "TI-Boost"
- note removed: "USB-A"
- note removed: "Vbatt"
- note removed: "Vbus"
- note removed: "resistor values are specific to iOS -\n to charge other devices, \nchange values accordingly"
- moved on the sheet: C2, C3, D1, D2, F1, J1, J2, R11, R12, R13, R5, R6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
