File: hv_power_supply/power_bank/Antoinette_power_bank/Antoinette_PowerBank.sch (KiCad schematic (older format))
At the start: 43 parts, among them J1 CONN_01x02, J2 USB_A, J3 CONN_01x02, Q1 SSM3K333R, U1 USB_MicroB, U2 MCP73871T-2CCI_ML, U3 TPS61090RSAR

Commit message: changed +batt to VBATT and created initial layout for power bank
Parts:
- removed J1, J3: CONN_01x02, Connector_PinHeader_2.54mm:PinHeader_1x02_P2.54mm_Vertical, symbol formula:CONN_01x02
- removed J2: USB_A, symbol formula:USB_A
- removed U1: USB_MicroB, Connectors_USB:USB_Micro-B_Molex-105017-0001, symbol formula:USB_MicroB
- added J1, J3: NanoFit_RA_TH_02, footprints:NanoFit_Molex_1x02x2.50mm_Angled_OEM, symbol formula:NanoFit_RA_TH_02
- added J2: USB-Micro-1981568-1, footprints:TE_1981568-1, symbol formula:USB-Micro-1981568-1
- added J4: USB-A-S-X-X-SM2, footprints:SAMTEC_USB-A-S-X-X-SM2, symbol formula:USB-A-S-X-X-SM2
- C7: footprint footprints:C_1812_OEM -> footprints:C_1812_4532Metric
- L1: footprint (none) -> footprints:L_100uH_OEM
Connections:
- net labels removed: +BATT
- wire segments 106 -> 108
Other:
- moved on the sheet: C1, C2, F1, R1, R17, R18, R2, TP1

Commit message: modify schematic to be pull up resistor for LBO pin and update PCB layout to fit DXF
Parts:
- C1, C2, C4: symbol formula:C_10uF -> Antoinette_PowerBank-rescue:C_10uF-formula
- C3: symbol formula:C_10nF -> Antoinette_PowerBank-rescue:C_10nF-formula
- C5: symbol formula:C_0.1uF -> Antoinette_PowerBank-rescue:C_0.1uF-formula
- C6: symbol formula:C_2.2uF -> Antoinette_PowerBank-rescue:C_2.2uF-formula
- C7: symbol formula:C_100uF -> Antoinette_PowerBank-rescue:C_100uF-formula
- D1: symbol formula:LED_0805_Amber -> Antoinette_PowerBank-rescue:LED_0805_Amber-formula
- D2, D3, D4: symbol formula:LED_0805 -> Antoinette_PowerBank-rescue:LED_0805-formula
- F1: symbol formula:1.5A_Fuse -> Antoinette_PowerBank-rescue:1.5A_Fuse-formula
- J1, J3: symbol formula:NanoFit_RA_TH_02 -> Antoinette_PowerBank-rescue:NanoFit_RA_TH_02-formula
- J2: symbol formula:USB-Micro-1981568-1 -> Antoinette_PowerBank-rescue:USB-Micro-1981568-1-formula
- J4: symbol formula:USB-A-S-X-X-SM2 -> Antoinette_PowerBank-rescue:USB-A-S-X-X-SM2-formula
- L1: symbol formula:L_6.8uH -> Antoinette_PowerBank-rescue:L_6.8uH-formula
- Q1: symbol formula:SSM3K333R -> Antoinette_PowerBank-rescue:SSM3K333R-formula
- R1: symbol formula:R_75k -> Antoinette_PowerBank-rescue:R_75k-formula
- R10, R13: symbol formula:R_200K -> Antoinette_PowerBank-rescue:R_200K-formula
- R11, R15, R16, R8, R9: symbol formula:R_1K -> Antoinette_PowerBank-rescue:R_1K-formula
- R12, R6: symbol formula:R_1.87M -> Antoinette_PowerBank-rescue:R_1.87M-formula
- R14: symbol formula:R_10K -> Antoinette_PowerBank-rescue:R_10K-formula
- R17: symbol formula:R_43k -> Antoinette_PowerBank-rescue:R_43k-formula
- R18, R2: symbol formula:R_49.9K -> Antoinette_PowerBank-rescue:R_49.9K-formula
- R3: symbol formula:R_270K -> Antoinette_PowerBank-rescue:R_270K-formula
- R4, R5: symbol formula:R_100K -> Antoinette_PowerBank-rescue:R_100K-formula
- R7: symbol formula:R_340K -> Antoinette_PowerBank-rescue:R_340K-formula
- TP1, TP2, TP3, TP4, TP5: symbol formula:TP -> Antoinette_PowerBank-rescue:TP-formula
- U2: symbol formula:MCP73871T-2CCI_ML -> Antoinette_PowerBank-rescue:MCP73871T-2CCI_ML-formula
- U3: symbol formula:TPS61090RSAR -> Antoinette_PowerBank-rescue:TPS61090RSAR-formula
Connections:
- net +5V: now also R14.1, R15.1
- net +BATT: no longer R15.1
- net GND: no longer R14.2
- net at Q1.1 (G), TP5.1 (TP), U3.12 (LBO): now also R14.2; no longer R14.1
Other:
- moved on the sheet: R14
