File: hv_power_supply/power_bank/Antoinette_power_bank/Antoinette_PowerBank.sch (KiCad schematic (older format))
At the start: 44 parts, among them J1 NanoFit_RA_TH_02, J2 USB-Micro-1981568-1, J3 NanoFit_RA_TH_02, J4 USB-A-S-X-X-SM2, J5 NanoFit_RA_TH_02, Q1 SSM3K333R, U2 MCP73871T-2CCI_ML, U3 TPS61090RSAR

Commit message: fixed library typos and adjusted silkscreen
Parts:
- C1, C2, C4: symbol Formula:C_10uF -> formula:C_10uF
- C3: symbol Formula:C_10nF -> formula:C_10nF
- C5: symbol Formula:C_0.1uF -> formula:C_0.1uF
- C6: symbol Formula:C_2.2uF -> formula:C_2.2uF
- C7: symbol Formula:C_100uF -> formula:C_100uF
- D1: symbol Formula:LED_0805_Amber -> formula:LED_0805_Amber
- D2, D3, D4: symbol Formula:LED_0805 -> formula:LED_0805
- F1: symbol Formula:1.5A_Fuse -> formula:1.5A_Fuse
- J1: symbol Formula:NanoFit_RA_TH_02 -> formula:NanoFit_RA_TH_02
- J2: symbol Formula:USB-Micro-1981568-1 -> formula:USB-Micro-1981568-1
- J3, J5: footprint Formula:NanoFit_Molex_1x02x2.50mm_Angled_OEM -> formula:NanoFit_Molex_1x02x2.50mm_Angled_OEM; symbol Formula:NanoFit_RA_TH_02 -> formula:NanoFit_RA_TH_02
- J4: symbol Formula:USB-A-S-X-X-SM2 -> formula:USB-A-S-X-X-SM2
- L1: symbol Formula:L_6.8uH -> formula:L_6.8uH
- Q1: symbol Formula:SSM3K333R -> formula:SSM3K333R
- R1: symbol Formula:R_75k -> formula:R_75k
- R10, R13: symbol Formula:R_200K -> formula:R_200K
- R11, R8, R9: symbol Formula:R_1K -> formula:R_1K
- R12, R6: symbol Formula:R_1.87M -> formula:R_1.87M
- R14: symbol Formula:R_10K -> formula:R_10K
- R15, R16: symbol Formula:R_330 -> formula:R_330
- R17: symbol Formula:R_43k -> formula:R_43k
- R18, R2: symbol Formula:R_49.9K -> formula:R_49.9K
- R3: symbol Formula:R_270K -> formula:R_270K
- R4, R5: symbol Formula:R_100K -> formula:R_100K
- R7: symbol Formula:R_340K -> formula:R_340K
- TP1, TP2, TP3, TP4, TP5: symbol Formula:TP -> formula:TP
- U2: symbol Formula:MCP73871T-2CCI_ML -> formula:MCP73871T-2CCI_ML
- U3: symbol Formula:TPS61090RSAR -> formula:TPS61090RSAR
Changed lines of the file:
@@
 $EndDescr
 $Comp
-L Formula:1.5A_Fuse F1
+L formula:1.5A_Fuse F1
 U 1 1 5F921D2E
 P 2000 3950
@@
 	2450 1550 2450 1350
 $Comp
-L Formula:C_10uF C1
+L formula:C_10uF C1
 U 1 1 5F924127
 P 2450 2100
@@
 	2450 1900 2450 1550
 $Comp
-L Formula:R_49.9K R2
+L formula:R_49.9K R2
 U 1 1 5F924143
 P 2950 2100
@@
      Output USB\n(to charge phone)
 $Comp
-L Formula:R_75k R1
+L formula:R_75k R1
 U 1 1 5F924176
 P 2950 1400
@@
 Input USB\n(to charge bat)
 $Comp
-L Formula:C_10uF C2
+L formula:C_10uF C2
 U 1 1 5F92E826
 P 1950 5400
@@
 NoConn ~ 1500 5250
 $Comp
-L Formula:TP TP1
+L formula:TP TP1
 U 1 1 5F936478
 P 1700 4950
@@
 $EndComp
 $Comp
-L Formula:TPS61090RSAR U3
+L formula:TPS61090RSAR U3
 U 1 1 5F93A0E2
 P 7900 1800
@@
 $EndComp
 $Comp
-L Formula:L_6.8uH L1
+L formula:L_6.8uH L1
 U 1 1 5F93B925
 P 6850 1500
@@
 	7200 1500 6950 1500
 $Comp
-L Formula:TP TP3
+L formula:TP TP3
 U 1 1 5F93E0BD
 P 6000 1300
@@
 $EndComp
 $Comp
-L Formula:VBATT #PWR016
+L formula:VBATT #PWR016
 U 1 1 5F94059A
 P 5700 1450
@@
 	7200 1600 7200 1500
 $Comp
-L Formula:TP TP4
+L formula:TP TP4
 U 1 1 5F94306C
 P 2500 6600
@@
 $EndComp
 $Comp
-L Formula:R_200K R10
+L formula:R_200K R10
 U 1 1 5F9446C9
 P 2450 6450
@@
 	2600 6450 2800 6450
 $Comp
-L Formula:C_0.1uF C5
+L formula:C_0.1uF C5
 U 1 1 5F94A827
 P 6050 1950
@@
 $EndComp
 $Comp
-L Formula:C_10uF C4
+L formula:C_10uF C4
 U 1 1 5F94B212
 P 5700 2000
@@
 $EndComp
 $Comp
-L Formula:R_340K R7
+L formula:R_340K R7
 U 1 1 5F94FB34
 P 6300 2450
@@
 	8700 1700 8750 1700
 $Comp
-L Formula:C_2.2uF C6
+L formula:C_2.2uF C6
 U 1 1 5F912C95
 P 9350 1750
@@
 	10500 1400 10500 1500
 $Comp
-L Formula:LED_0805 D4
+L formula:LED_0805 D4
 U 1 1 5F927053
 P 10500 1950
@@
 	10500 2200 10500 2100
 $Comp
-L Formula:R_200K R13
+L formula:R_200K R13
 U 1 1 5F929ECA
 P 9000 2050
@@
 	8600 1900 9000 1900
 $Comp
-L Formula:R_1.87M R12
+L formula:R_1.87M R12
 U 1 1 5F93C0EB
 P 9000 1700
@@
 	9000 1850 9000 1900
 $Comp
-L Formula:TP TP5
+L formula:TP TP5
 U 1 1 5F942010
 P 9100 2950
@@
 $EndComp
 $Comp
-L Formula:R_10K R14
+L formula:R_10K R14
 U 1 1 5F943142
 P 9300 3000
@@
 $EndComp
 $Comp
-L Formula:SSM3K333R Q1
+L formula:SSM3K333R Q1
 U 1 1 5F9440B8
 P 9600 3150
@@
 $EndComp
 $Comp
-L Formula:LED_0805 D3
+L formula:LED_0805 D3
 U 1 1 5F94621C
 P 9700 2800
@@
 	6850 4450 6850 4200
 $Comp
-L Formula:LED_0805 D2
+L formula:LED_0805 D2
 U 1 1 5F9F9473
 P 6950 4550
@@
 $EndComp
 $Comp
-L Formula:R_1K R11
+L formula:R_1K R11
 U 1 1 5F9FB8C1
 P 7250 4550
@@
 	7550 4550 7400 4550
 $Comp
-L Formula:R_100K R5
+L formula:R_100K R5
 U 1 1 5FA06FD7
 P 6100 5600
@@
 	6100 5350 6100 5450
 $Comp
-L Formula:R_1K R9
+L formula:R_1K R9
 U 1 1 5FA09BF6
 P 6550 5550
@@
 	3800 4050 3950 4050
 $Comp
-L Formula:R_270K R3
+L formula:R_270K R3
 U 1 1 5FA207E3
 P 3800 3900
@@
 	3950 4050 3950 4450
 $Comp
-L Formula:R_100K R4
+L formula:R_100K R4
 U 1 1 5FA2A403
 P 3800 4200
@@
 $EndComp
 $Comp
-L Formula:TP TP2
+L formula:TP TP2
 U 1 1 5FA387DD
 P 3800 4950
@@
 	3600 5150 3600 5050
 $Comp
-L Formula:C_10nF C3
+L formula:C_10nF C3
 U 1 1 5FA5B66D
 P 3800 5500
@@
 Battery + Load Manager
 $Comp
-L Formula:R_43k R17
+L formula:R_43k R17
 U 1 1 5FAC4418
 P 3500 1400
@@
 $EndComp
 $Comp
-L Formula:R_49.9K R18
+L formula:R_49.9K R18
 U 1 1 5FAEF9FD
 P 3500 2100
@@
 	3500 2400 3500 2250
 $Comp
-L Formula:LED_0805_Amber D1
+L formula:LED_0805_Amber D1
 U 1 1 5F9F302E
 P 6200 4450
@@
 	6800 4550 5650 4550
 $Comp
-L Formula:R_1K R8
+L formula:R_1K R8
 U 1 1 5F9F422E
 P 6500 4450
@@
 $EndComp
 $Comp
-L Formula:VBATT #PWR015
+L formula:VBATT #PWR015
 U 1 1 5F9ED162
 P 5650 4000
@@
 $EndComp
 $Comp
-L Formula:MCP73871T-2CCI_ML U2
+L formula:MCP73871T-2CCI_ML U2
 U 1 1 5F9E9E16
 P 4850 4950
@@
 Power Bank Project
 $Comp
-L Formula:USB-A-S-X-X-SM2 J4
+L formula:USB-A-S-X-X-SM2 J4
 U 1 1 5FB17265
 P 1900 1750
@@
 	1500 5750 1650 5750
 $Comp
-L Formula:USB-Micro-1981568-1 J2
+L formula:USB-Micro-1981568-1 J2
 U 1 1 5FB0DC42
 P 1200 5450
@@
 	2300 2200 2450 2200
 $Comp
-L Formula:C_100uF C7
+L formula:C_100uF C7
 U 1 1 5FBD94B6
 P 9700 1700
@@
 $EndComp
 $Comp
-L Formula:NanoFit_RA_TH_02 J1
+L formula:NanoFit_RA_TH_02 J1
 U 1 1 5FB78F91
 P 1100 2850
@@
 $EndComp
 $Comp
-L Formula:NanoFit_RA_TH_02 J3
+L formula:NanoFit_RA_TH_02 J3
 U 1 1 5FBCFFB4
 P 1250 4050
 F 0 "J3" H 1142 3663 60  0000 C CNN
 F 1 "NanoFit_RA_TH_02" H 1142 3769 60  0000 C CNN
-F 2 "Formula:NanoFit_Molex_1x02x2.50mm_Angled_OEM" H 1250 3450 60  0001 C CNN
+F 2 "formula:NanoFit_Molex_1x02x2.50mm_Angled_OEM" H 1250 3450 60  0001 C CNN
 F 3 "https://www.molex.com/pdm_docs/sd/1053131102_sd.pdf" H 1250 3600 60  0001 C CNN
 F 4 "DK" H 1250 4600 50  0001 C CNN "MFN"
@@
 $EndComp
 $Comp
-L Formula:R_1.87M R6
+L formula:R_1.87M R6
 U 1 1 5FC80133
 P 6300 1950
@@
 $EndComp
 $Comp
-L Formula:VBATT #PWR0102
+L formula:VBATT #PWR0102
 U 1 1 5FCBCBA4
 P 2800 6450
@@
 switch
 $Comp
-L Formula:NanoFit_RA_TH_02 J5
+L formula:NanoFit_RA_TH_02 J5
 U 1 1 6034D59C
 P 1700 6550
 F 0 "J5" H 1592 6163 60  0000 C CNN
 F 1 "NanoFit_RA_TH_02" H 1592 6269 60  0000 C CNN
-F 2 "Formula:NanoFit_Molex_1x02x2.50mm_Angled_OEM" H 1700 5950 60  0001 C CNN
+F 2 "formula:NanoFit_Molex_1x02x2.50mm_Angled_OEM" H 1700 5950 60  0001 C CNN
 F 3 "https://www.molex.com/pdm_docs/sd/1053131102_sd.pdf" H 1700 6100 60  0001 C CNN
 F 4 "DK" H 1700 7100 50  0001 C CNN "MFN"
@@
 	8600 1550 8600 1450
 $Comp
-L Formula:R_330 R16
+L formula:R_330 R16
 U 1 1 60365C24
 P 10500 1650
@@
 $EndComp
 $Comp
-L Formula:R_330 R15
+L formula:R_330 R15
 U 1 1 6036A43B
 P 9700 2500

Commit message: make silkscreen more legible
Parts:
- J3, J5: footprint formula:NanoFit_Molex_1x02x2.50mm_Angled_OEM -> footprints:NanoFit_Molex_1x02x2.50mm_Angled_OEM
Changed lines of the file:
@@
-$EndComp
-$Comp
-L formula:NanoFit_RA_TH_02 J3
-U 1 1 5FBCFFB4
-P 1250 4050
-F 0 "J3" H 1142 3663 60  0000 C CNN
-F 1 "NanoFit_RA_TH_02" H 1142 3769 60  0000 C CNN
-F 2 "formula:NanoFit_Molex_1x02x2.50mm_Angled_OEM" H 1250 3450 60  0001 C CNN
-F 3 "https://www.molex.com/pdm_docs/sd/1053131102_sd.pdf" H 1250 3600 60  0001 C CNN
-F 4 "DK" H 1250 4600 50  0001 C CNN "MFN"
-F 5 "WM14972-ND" H 1250 4500 50  0001 C CNN "MPN"
-F 6 "https://www.digikey.com/products/en/connectors-interconnects/rectangular-connectors-headers-male-pins/314?k=nanofit+2&k=&pkeyword=nanofit+2&pv88=2&pv69=367&sf=0&FV=ffe0013a&quantity=&ColumnSort=0&page=1&pageSize=25" H 1250 3250 50  0001 C CNN "PurchasingLink"
-	1    1250 4050
-	-1   0    0    1
 $EndComp
 $Comp
@@
 Text Label 2150 6450 0    50   ~ 0
 switch
-$Comp
-L formula:NanoFit_RA_TH_02 J5
-U 1 1 6034D59C
-P 1700 6550
-F 0 "J5" H 1592 6163 60  0000 C CNN
-F 1 "NanoFit_RA_TH_02" H 1592 6269 60  0000 C CNN
-F 2 "formula:NanoFit_Molex_1x02x2.50mm_Angled_OEM" H 1700 5950 60  0001 C CNN
-F 3 "https://www.molex.com/pdm_docs/sd/1053131102_sd.pdf" H 1700 6100 60  0001 C CNN
-F 4 "DK" H 1700 7100 50  0001 C CNN "MFN"
-F 5 "WM14972-ND" H 1700 7000 50  0001 C CNN "MPN"
-F 6 "https://www.digikey.com/products/en/connectors-interconnects/rectangular-connectors-headers-male-pins/314?k=nanofit+2&k=&pkeyword=nanofit+2&pv88=2&pv69=367&sf=0&FV=ffe0013a&quantity=&ColumnSort=0&page=1&pageSize=25" H 1700 5750 50  0001 C CNN "PurchasingLink"
-	1    1700 6550
-	-1   0    0    1
-$EndComp
 Wire Wire Line
 	1500 5150 1700 5150
@@
 	1    0    0    -1
 $EndComp
+$Comp
+L formula:NanoFit_RA_TH_02 J3
+U 1 1 60426277
+P 1250 4050
+F 0 "J3" H 1142 3663 60  0000 C CNN
+F 1 "NanoFit_RA_TH_02" H 1142 3769 60  0000 C CNN
+F 2 "footprints:NanoFit_Molex_1x02x2.50mm_Angled_OEM" H 1250 3450 60  0001 C CNN
+F 3 "https://www.molex.com/pdm_docs/sd/1053131102_sd.pdf" H 1250 3600 60  0001 C CNN
+F 4 "DK" H 1250 4600 50  0001 C CNN "MFN"
+F 5 "WM14972-ND" H 1250 4500 50  0001 C CNN "MPN"
+F 6 "https://www.digikey.com/products/en/connectors-interconnects/rectangular-connectors-headers-male-pins/314?k=nanofit+2&k=&pkeyword=nanofit+2&pv88=2&pv69=367&sf=0&FV=ffe0013a&quantity=&ColumnSort=0&page=1&pageSize=25" H 1250 3250 50  0001 C CNN "PurchasingLink"
+	1    1250 4050
+	-1   0    0    1
+$EndComp
+$Comp
+L formula:NanoFit_RA_TH_02 J5
+U 1 1 6042CE2F
+P 1700 6550
+F 0 "J5" H 1592 6163 60  0000 C CNN
+F 1 "NanoFit_RA_TH_02" H 1592 6269 60  0000 C CNN
+F 2 "footprints:NanoFit_Molex_1x02x2.50mm_Angled_OEM" H 1700 5950 60  0001 C CNN
+F 3 "https://www.molex.com/pdm_docs/sd/1053131102_sd.pdf" H 1700 6100 60  0001 C CNN
+F 4 "DK" H 1700 7100 50  0001 C CNN "MFN"
+F 5 "WM14972-ND" H 1700 7000 50  0001 C CNN "MPN"
+F 6 "https://www.digikey.com/products/en/connectors-interconnects/rectangular-connectors-headers-male-pins/314?k=nanofit+2&k=&pkeyword=nanofit+2&pv88=2&pv69=367&sf=0&FV=ffe0013a&quantity=&ColumnSort=0&page=1&pageSize=25" H 1700 5750 50  0001 C CNN "PurchasingLink"
+	1    1700 6550
+	-1   0    0    1
+$EndComp
 $EndSCHEMATC
