File: hv_power_supply/power_bank/Sushmit_Power_Bank/PowerBankSushmit1.sch (KiCad schematic (older format))
At the start: 48 parts, among them J1 CONN_01x02, J2 CONN_01x02, J3 USB_A, Q1 SSM3K333R, U1 USB_MicroB, U2 MCP73871T-2CCI_ML-formula, U3 TPS61090RSAR-formula

Commit message: DIY PowerBankSushmit1 - Changing library names
Parts:
- C1, C2, C3, C4, C6, C7: symbol AdvancedResarch:C_10uF-formula -> formula:C_10uF-formula
- C5: symbol AdvancedResarch:C_10nF-formula -> formula:C_10nF-formula
- D1, D3, D4: symbol AdvancedResarch:LED_0805-formula -> formula:LED_0805-formula
- D2: symbol AdvancedResarch:LED_0805_Amber-formula -> formula:LED_0805_Amber-formula
- F1: symbol AdvancedResarch:1.5A_Fuse-formula -> formula:1.5A_Fuse-formula
- J1, J2: symbol AdvancedResarch:CONN_01x02-formula -> formula:CONN_01x02-formula
- L1: symbol AdvancedResarch:L_6.8uH-formula -> formula:L_6.8uH-formula
- Q1: symbol AdvancedResarch:SSM3K333R-formula -> formula:SSM3K333R-formula
- R1, R10, R11, R12, R13, R14, R15, R16, R17, R18, R2, R3, R4, R5, R6, R7, R8, R9: symbol AdvancedResearch:formula_R_1K -> formula:formula_R_1K
- TP1, TP2, TP3, TP4, TP5: symbol AdvancedResarch:TP-formula -> formula:TP-formula
- U1: symbol AdvancedResarch:USB_MicroB-formula -> formula:USB_MicroB-formula
- U2: symbol AdvancedResarch:MCP73871T-2CCI_ML-formula -> formula:MCP73871T-2CCI_ML-formula
- U3: symbol AdvancedResarch:TPS61090RSAR-formula -> formula:TPS61090RSAR-formula
Changed lines of the file:
@@
 $EndComp
 $Comp
-L AdvancedResearch:formula_R_1K R1
+L formula:formula_R_1K R1
 U 1 1 5F8DBFCA
 P 3050 1650
@@
 $EndComp
 $Comp
-L AdvancedResearch:formula_R_1K R3
+L formula:formula_R_1K R3
 U 1 1 5F8DE663
 P 3800 1650
@@
 $EndComp
 $Comp
-L AdvancedResearch:formula_R_1K R4
+L formula:formula_R_1K R4
 U 1 1 5F8DED9A
 P 3800 2800
@@
 $EndComp
 $Comp
-L AdvancedResearch:formula_R_1K R2
+L formula:formula_R_1K R2
 U 1 1 5F8DF8D7
 P 3050 2800
@@
 	2200 1950 2500 1950
 $Comp
-L AdvancedResarch:C_10uF-formula C1
+L formula:C_10uF-formula C1
 U 1 1 5F8E35C6
 P 2500 2600
@@
 Thermistor\n
 $Comp
-L AdvancedResarch:CONN_01x02-formula J1
+L formula:CONN_01x02-formula J1
 U 1 1 5F8F0921
 P 1775 3525
@@
 Battery\n
 $Comp
-L AdvancedResarch:CONN_01x02-formula J2
+L formula:CONN_01x02-formula J2
 U 1 1 5F8FB661
 P 3075 3525
@@
 $EndComp
 $Comp
-L AdvancedResarch:1.5A_Fuse-formula F1
+L formula:1.5A_Fuse-formula F1
 U 1 1 5F8FC8AA
 P 3675 3525
@@
 Input USB\n(To charge bat)\n
 $Comp
-L AdvancedResarch:USB_MicroB-formula U1
+L formula:USB_MicroB-formula U1
 U 1 1 5F904C79
 P 1950 5050
@@
 $EndComp
 $Comp
-L AdvancedResarch:C_10uF-formula C2
+L formula:C_10uF-formula C2
 U 1 1 5F907617
 P 3300 5150
@@
 $EndComp
 $Comp
-L AdvancedResarch:TP-formula TP2
+L formula:TP-formula TP2
 U 1 1 5F908C0C
 P 2800 4650
@@
 $EndComp
 $Comp
-L AdvancedResarch:TP-formula TP1
+L formula:TP-formula TP1
 U 1 1 5F99B72A
 P 9250 2975
@@
 	7000 1425 7000 1525
 $Comp
-L AdvancedResarch:TP-formula TP4
+L formula:TP-formula TP4
 U 1 1 5F9CCC74
 P 6600 1825
@@
 $EndComp
 $Comp
-L AdvancedResearch:formula_R_1K R9
+L formula:formula_R_1K R9
 U 1 1 5F9ED429
 P 6700 1975
@@
 $EndComp
 $Comp
-L AdvancedResearch:formula_R_1K R6
+L formula:formula_R_1K R6
 U 1 1 5F9D46E3
 P 6200 2325
@@
 $EndComp
 $Comp
-L AdvancedResearch:formula_R_1K R5
+L formula:formula_R_1K R5
 U 1 1 5F9D32FD
 P 6200 1875
@@
 $EndComp
 $Comp
-L AdvancedResarch:C_10uF-formula C4
+L formula:C_10uF-formula C4
 U 1 1 5F9D1F1C
 P 5800 1925
@@
 $EndComp
 $Comp
-L AdvancedResarch:C_10uF-formula C3
+L formula:C_10uF-formula C3
 U 1 1 5F9CFEE1
 P 5350 1925
@@
 $EndComp
 $Comp
-L AdvancedResarch:VBATT-formula #PWR0119
+L formula:VBATT-formula #PWR0119
 U 1 1 5F9CDDDA
 P 5350 1375
@@
 $EndComp
 $Comp
-L AdvancedResarch:TP-formula TP3
+L formula:TP-formula TP3
 U 1 1 5F9CBEC6
 P 5850 1225
@@
 $EndComp
 $Comp
-L AdvancedResarch:L_6.8uH-formula L1
+L formula:L_6.8uH-formula L1
 U 1 1 5F9C9CAD
 P 6600 1425
@@
 $EndComp
 $Comp
-L AdvancedResarch:GNDPWR-formula #PWR0121
+L formula:GNDPWR-formula #PWR0121
 U 1 1 5F9C1E1E
 P 8000 2625
@@
 $EndComp
 $Comp
-L AdvancedResarch:GNDPWR-formula #PWR0122
+L formula:GNDPWR-formula #PWR0122
 U 1 1 5F9BE2AC
 P 8400 1675
@@
 $EndComp
 $Comp
-L AdvancedResarch:GNDPWR-formula #PWR0123
+L formula:GNDPWR-formula #PWR0123
 U 1 1 5F9BD705
 P 8400 2275
@@
 $EndComp
 $Comp
-L AdvancedResarch:LED_0805-formula D4
+L formula:LED_0805-formula D4
 U 1 1 5F9B7FA3
 P 10350 1675
@@
 $EndComp
 $Comp
-L AdvancedResarch:LED_0805-formula D3
+L formula:LED_0805-formula D3
 U 1 1 5F9B3FDB
 P 10100 2575
@@
 	8400 1375 8400 1425
 $Comp
-L AdvancedResarch:C_10uF-formula C7
+L formula:C_10uF-formula C7
 U 1 1 5F98B3BA
 P 9900 1625
@@
 $EndComp
 $Comp
-L AdvancedResarch:C_10uF-formula C6
+L formula:C_10uF-formula C6
 U 1 1 5F989D80
 P 9450 1625
@@
 $EndComp
 $Comp
-L AdvancedResearch:formula_R_1K R16
+L formula:formula_R_1K R16
 U 1 1 5F987A2C
 P 10100 2275
@@
 $EndComp
 $Comp
-L AdvancedResearch:formula_R_1K R18
+L formula:formula_R_1K R18
 U 1 1 5F98700B
 P 10350 1375
@@
 $EndComp
 $Comp
-L AdvancedResearch:formula_R_1K R12
+L formula:formula_R_1K R12
 U 1 1 5F9868B2
 P 9000 2025
@@
 $EndComp
 $Comp
-L AdvancedResearch:formula_R_1K R11
+L formula:formula_R_1K R11
 U 1 1 5F985E27
 P 9000 1575
@@
 NoConn ~ 7950 4800
 $Comp
-L AdvancedResarch:C_10nF-formula C5
+L formula:C_10nF-formula C5
 U 1 1 5F8DA1C5
 P 5850 5550
@@
 	1100 6100 6025 6100
 $Comp
-L AdvancedResearch:formula_R_1K R15
+L formula:formula_R_1K R15
 U 1 1 5F988D3D
 P 9650 3325
@@
 $EndComp
 $Comp
-L AdvancedResarch:SSM3K333R-formula Q1
+L formula:SSM3K333R-formula Q1
 U 1 1 5F9AF6F7
 P 10000 3175
@@
 $EndComp
 $Comp
-L AdvancedResearch:formula_R_1K R7
+L formula:formula_R_1K R7
 U 1 1 5F9273DC
 P 5650 3750
@@
 Battery+
 $Comp
-L AdvancedResarch:MCP73871T-2CCI_ML-formula U2
+L formula:MCP73871T-2CCI_ML-formula U2
 U 1 1 5F910070
 P 7150 5000
@@
 $EndComp
 $Comp
-L AdvancedResarch:VBATT-formula #PWR0131
+L formula:VBATT-formula #PWR0131
 U 1 1 5F91560A
 P 8100 4150
@@
 $EndComp
 $Comp
-L AdvancedResarch:LED_0805_Amber-formula D2
+L formula:LED_0805_Amber-formula D2
 U 1 1 5F917D3C
 P 8600 4500
@@
 $EndComp
 $Comp
-L AdvancedResearch:formula_R_1K R13
+L formula:formula_R_1K R13
 U 1 1 5F919491
 P 8900 4500
@@
 $EndComp
 $Comp
-L AdvancedResarch:LED_0805-formula D1
+L formula:LED_0805-formula D1
 U 1 1 5F91B1B0
 P 9550 4600
@@
 $EndComp
 $Comp
-L AdvancedResearch:formula_R_1K R17
+L formula:formula_R_1K R17
 U 1 1 5F91EA7B
 P 9850 4600
@@
 $EndComp
 $Comp
-L AdvancedResearch:formula_R_1K R10
+L formula:formula_R_1K R10
 U 1 1 5F9213A6
 P 8400 5700
@@
 $EndComp
 $Comp
-L AdvancedResearch:formula_R_1K R14
+L formula:formula_R_1K R14
 U 1 1 5F922E1F
 P 9100 5700
@@
 Connection ~ 6350 5400
 $Comp
-L AdvancedResarch:TP-formula TP5
+L formula:TP-formula TP5
 U 1 1 5F95154A
 P 5800 5050
@@
 $EndComp
 $Comp
-L AdvancedResearch:formula_R_1K R8
+L formula:formula_R_1K R8
 U 1 1 5F923688
 P 5650 4200
@@
 	8400 1825 9000 1825
 $Comp
-L AdvancedResarch:TPS61090RSAR-formula U3
+L formula:TPS61090RSAR-formula U3
 U 1 1 5F983A4C
 P 7700 1725
