File: firmware_revamp/boards/abitamim_project/Proto1/Proto1.sch (KiCad schematic (older format))
At the start: 42 parts, among them J1 CONN_02X03, U1 HC-05, U1 MCP2561-E_SN, U2 ATMEGA16M1, Y1 Crystal_SMD

Commit message: Adding my arduino board proto 1
Parts:
- gave numbers to parts that had none: 29
- renumbered C2 to C1, C1 to C12, C3 to C2, C4 to C5, C5 to C8, J1 to J3, R2 to R12, R3 to R6, U1 to U5, U1 to U6
Connections:
- net labels removed: 12V, 3V3, 5V, CAN_Rx, CAN_Tx, VCC
- no-connect marks 2 -> 42
