File: firmware_revamp/boards/bEnJi_ArDuInO/benji_arduino2.sch (KiCad schematic (older format))
At the start: 36 parts

Commit message: removed erroneous add to telemetry, added working schematic to firmware
Parts:
- added C12: C_30pF, footprints:C_0805_OEM, symbol formula:C_30pF
- added C5: C_0.1uF, footprints:C_0805_OEM, symbol formula:C_0.1uF
- J1: renamed from J?; symbol Connector:USB_B -> benji_arduino2-rescue:USB_B-Connector
- gave numbers to parts that had none: 35
Connections:
- net labels added: AREF
- wire segments 93 -> 105
- no-connect marks 11 -> 13
