File: hardware_in_the_loop/boards/agnostic_testing_board/agnostic_testing_board.sch (KiCad schematic (older format))
At the start: 44 parts, among them J1 CONN_02X03, U1 MCP2561-E_SN, U2 ATMEGA16M1, Y1 Crystal_SMD

Commit message: Emily's Schematic second draft - for review
Parts:
- removed Q? (x2): SSM3K333R, footprints:SOT-23F, symbol formula:SSM3K333R
- added C?: C_10nF, footprints:C_0805_OEM, symbol formula:C_10nF
- added C?: C_100nF, footprints:C_0603_1608Metric, symbol formula:C_100nF
- added F?: F_500mA_16V, footprints:Fuse_1210, symbol formula:F_500mA_16V
- added J?: INPUT_POWER_CONNECTOR_PLACEHOLDER, symbol formula:Ampseal_08_RA
- added K? (x2): G5Q-1A4-DC12, footprints:Relay_SPST_OMRON-G5Q-1A4_OEM, symbol formula:G5Q-1A4-DC12
- added R? (x8): R_1K, footprints:R_0805_OEM, symbol formula:R_1K
Connections:
- net BRAKELIGHT_LSD is gone; now on net LSD_1: J?.13
- net BSPD_RELAY_LSD is gone; now on net LSD_2: J?.17
- net GND: now also J?.10, J?.11, J?.6, C?.2, K?.5, K?.5, R?.1, R?.1, R?.1; no longer J?.5 (Shield)
- net VCC: now also C?.1, R?.1, R?.1
- net at U2.17 ((PCINT12/ADC8/ACMPN3/AMP1-)PC4): now also R?.2
- net at U2.18 ((PCINT13/ADC9/ACMP3/AMP1+)PC5): now also R?.2
- net LSD_1: now reaches U2.22 ((PCINT14/ADC10/ACMP1)PC6)
- net LSD_1: now also J?.1, R?.2; no longer R?.2
- net LSD_2: now reaches U2.25 ((PCINT15/D2A/AMP2+)PC7)
- net LSD_2: now also R?.2; no longer R?.2
- net at U2.29 ((PCINT16/PSCOUT0A)PD0): now also R?.2, R?.2
- net at U2.32 ((PCINT17/CLKO/PSCIN0)PD1): now also R?.2, R?.2
- net Final_Shutdown: now reaches J?.12
- net Final_Shutdown: now also J?.2, R?.1
- net Air+Aux+: now reaches J?.3
- net Air+Aux+: now also K?.2
- net Air+Aux-: now reaches J?.4
- net Air+Aux-: now also K?.3
- net Air+Coll+: now reaches J?.5
- net Air+Coll+: now also R?.1
- net Air-Aux+: now reaches J?.7
- net Air-Aux+: now also K?.2
- net Air-Aux-: now reaches J?.8
- net Air-Aux-: now also K?.3
- net Air-Coll+: now reaches J?.9
- net Air-Coll+: now also R?.1
- new net: C?.1, F?.2, J?.1 (VBUS)
- new net: F?.1, U?.20 (VCC)
- new net: C?.2, U?.4 (VCCIO)
- new net 12v: J?.1
- new net not_enough_connectors_ATmega16: K?.1, K?.1, R?.2, R?.2
- no-connect marks 9 -> 5
Other:
- note added: "12V CONNECTOR PLACEHOLDER\n"
- note added: "Connectors\n"
- note added: "PINLESS COMPONENTS"
- note added: "To be replaced by correct connector after DR\n"
- note added: "USB TO FTDI\n"
- note removed: "2"
- moved on the sheet: C1, C2, C3, C4, C5, C?, D?, J1, J?, R1, R2, R3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
