File: hardware_in_the_loop/boards/Sensing_Suite_HITL/Sensing/Sensing.sch (KiCad schematic (older format))
At the start: 29 parts, among them J1 CONN_02X03, U1 MCP2561-E_SN, U101 TPS560430YF, U2 ATMEGA16M1, Y1 Crystal_SMD

Commit message: Updates to Template Board
Parts:
- added J?: Ampseal_23_VT, footprints:Ampseal_23, symbol formula:Ampseal_23_VT
- added J?: NanoFit_RA_TH_06, footprints:NanoFit_RA_6, symbol formula:NanoFit_RA_TH_06
- added J? (x12): MicroFit_V_2, footprints:MicroFit_V_2, symbol formula:MicroFit_V_2
- added U? (x2): 74HCT4051, symbol 74xx:74HCT4051
Connections:
- net 12V: now also J?.15, J?.17, J?.2, J?.21, J?.6
- net GND: now also J?.1, J?.12, J?.16, J?.18, J?.22, J?.3, J?.6, J?.7
- net MISO: now also J?.2
- net MOSI: now also J?.3
- net SCK: now also J?.4
- new net CAN_N: J?.11, J?.14, J?.20, J?.5
- new net CAN_P: J?.10, J?.13, J?.19, J?.4
- new net HALL_EFFECT_+: J?.1
- new net HALL_EFFECT_SENSE: J?.9
- new net LINEAR_POT_+: J?.8
- new net LINEAR_POT_-: J?.23
- new net SS: J?.5
- new net STRAIN_GAUGE_10_-: J?.2
- new net STRAIN_GAUGE_11_-: J?.2
- new net STRAIN_GAUGE_12_-: J?.2
- new net STRAIN_GAUGE_1_-: J?.2
- new net STRAIN_GAUGE_2_-: J?.2
- new net STRAIN_GAUGE_3_-: J?.2
- new net STRAIN_GAUGE_4_-: J?.2
- new net STRAIN_GAUGE_5_-: J?.2
- new net STRAIN_GAUGE_6_-: J?.2
- new net STRAIN_GAUGE_7_-: J?.2
- new net STRAIN_GAUGE_8_-: J?.2
- new net STRAIN_GAUGE_9_-: J?.2
- new net STRAIN_GUAGE_10_+: J?.1
- new net STRAIN_GUAGE_11_+: J?.1
- new net STRAIN_GUAGE_12_+: J?.1
- new net STRAIN_GUAGE_1_+: J?.1
- new net STRAIN_GUAGE_2_+: J?.1
- new net STRAIN_GUAGE_3_+: J?.1
- new net STRAIN_GUAGE_4_+: J?.1
- new net STRAIN_GUAGE_5_+: J?.1
- new net STRAIN_GUAGE_6_+: J?.1
- new net STRAIN_GUAGE_7_+: J?.1
- new net STRAIN_GUAGE_8_+: J?.1
- new net STRAIN_GUAGE_9_+: J?.1
Other:
- note added: "(CAN CABLE SHIELD)"

Commit message: Updates to Template Board
Other:
- note added: "*needs to be vertical (vt)"
Changed lines of the file:
@@
 Text Label 5900 6650 0    50   ~ 0
 STRAIN_GAUGE_9_-
+Text Notes 15050 5200 0    50   ~ 0
+*needs to be vertical (vt)
 $EndSCHEMATC

Commit message: Updates to the schematic
Parts:
- added J? (x2): MM_M_VT_08, footprints:micromatch_female_ra_8, symbol formula:MM_M_VT_08
- added J?: Ampseal_23_VT, footprints:Ampseal_23, symbol formula:Ampseal_23_VT
Connections:
- net labels added: HALL_EFFECT_-, LINEAR_POT_SENSE, STRAIN_GAUGE_1_+, STRAIN_GAUGE_2_+, STRAIN_GAUGE_MAIN, TO_DEMUX1A, TO_DEMUX1B, TO_DEMUX2A, TO_DEMUX2B
- wire segments 75 -> 79
Other:
- note added: "*before or\nafter demux"
- note added: "DEMUX1\n\n\n"
- note added: "DEMUX2\n\n"
- note added: "DIGITAL \nPOTENTIOMETER \nor \nRESISTOR DIVIDER\nfor Strain Gauge sensors"
- note added: "RC FILTER"
- note added: "Suspension Strain Gauge sensors\n"
- note added: "Suspension Travel Sensor"
- note added: "To Road Kill Harness\n\n"
- note added: "To Sensing Suite\n"
- note added: "Wheel Speed Sensor"
- moved on the sheet: J?, U?
