File: hv_power_supply/power_supply/buck_converter.sch (KiCad schematic (older format))
At the start: 0 parts

Commit message: HV Power Supply Buck Schematic (rev1)
Parts:
- added C_IN1: C_47uF, footprints:C_0805_OEM, symbol formula:C_47uF
- added C_OUT1: C_10uF, footprints:C_0805_OEM, symbol formula:C_10uF
- added DNP1, DNP2, DNP3: R_0, symbol Device:R
- added D_Schottky1: 10BQ100, symbol Device:D_Schottky
- added L_OUT1: L_10uH, symbol Device:L
- added R1: R_47k, symbol formula:R_47k
- added U1: TLF50211ELXUMA2, symbol formula:TLF50211ELXUMA2
Connections:
- net labels added: GND, VCC, VS
- wire segments 0 -> 36
Other:
- note added: "Input Cap 2"
- note added: "Input Cap 3\n"
- note added: "Input Inductor"
