File: hv_power_supply/power_supply/user_interface.sch (KiCad schematic (older format))
At the start: 0 parts

Commit message: user interface schematics
Parts:
- added C? (x2): C_30pF, footprints:C_0805_OEM, symbol formula:C_30pF
- added C?: C_0.1uF, footprints:C_0805_OEM, symbol formula:C_0.1uF
- added D? (x2): LED_0805, footprints:LED_0805_OEM, symbol formula:LED_0805
- added DS?: AMC1602AR-B-Y6WFDY-I2C, Display:HY1602E, symbol formula:AMC1602AR-B-Y6WFDY-I2C
- added J?: CONN_02X03, footprints:Pin_Header_Straight_2x03, symbol formula:CONN_02X03
- added R?: R_10K, footprints:R_0805_OEM, symbol formula:R_10K
- added R? (x3): R_200, footprints:R_0805_OEM, symbol formula:R_200
- added RV?: R_POT, symbol Device:R_POT
- added SW1?, SW?: EMS22A50-B28-LS6, symbol formula:EMS22A50-B28-LS6
- added U?: ATMEGA16M1, footprints:TQFP-32_7x7mm_Pitch0.8mm, symbol formula:ATMEGA16M1
- added Y?: Crystal_SMD, footprints:Crystal_SMD_FA238, symbol formula:Crystal_SMD
Connections:
- net labels added: CLK_I, CLK_V, CS_I, CS_V, D_OUTPUT_I, D_OUTPUT_V, GND, MISO, MOSI, PROGRAMMINGLED1, PROGRAMMINGLED2, RESET, SCK, SCL, SDA, VCC
- wire segments 0 -> 55
- no-connect marks 0 -> 3
Other:
- note added: "ATMEGA16M1\n"
- note added: "LCD DISPLAY\n"
- note added: "ROTARY ENCODER FOR CURRENT\n\n"
- note added: "ROTARY ENCODER FOR VOLTAGE\n"
