File: hv_power_supply/power_supply/user_interface.sch (KiCad schematic (older format))
At the start: 16 parts, among them SW1? EMS22A50-B28-LS6

Commit message: add hierarchical label and edit UI schematic
Parts:
- removed DS?: AMC1602AR-B-Y6WFDY-I2C, Display:HY1602E, symbol formula:AMC1602AR-B-Y6WFDY-I2C
- removed R?: R_200, footprints:R_0805_OEM, symbol formula:R_200
- removed RV?: R_POT, symbol Device:R_POT
- removed U?: ATMEGA16M1, footprints:TQFP-32_7x7mm_Pitch0.8mm, symbol formula:ATMEGA16M1
- added DS?: AMC1602AR-B-Y6WFDY-SPI, Display:HY1602E, symbol formula:AMC1602AR-B-Y6WFDY-SPI
- added R?: R_1.13K, footprints:R_0805_OEM, symbol formula:R_1.13K
- added R?: R_4.99K, footprints:R_0805_OEM, symbol formula:R_4.99K
- added U?: ATMEGA16M1, footprints:TQFP-32_7x7mm_Pitch0.8mm, symbol formula:ATMEGA16M1
Connections:
- net labels added: CLK, CS, CSB, OUTPUT_DAC, RS, SCLK, SID
- net labels removed: CLK_I, CLK_V, CS_I, CS_V, SCL, SDA
- wire segments 55 -> 53
- no-connect marks 3 -> 1
Other:
- moved on the sheet: C?, R?, SW1?, SW?, Y?

Commit message: edit schematics
Parts:
- added D? (x2): HLMP-Q150-F0011, footprints:HLMP-Q150-F0011, symbol formula:HLMP-Q150-F0011
- added R? (x2): R_3.01K, footprints:R_0805_OEM, symbol formula:R_3.01K
Connections:
- net labels added: DEBUG_LED1, DEBUG_LED2
- wire segments 53 -> 59
- no-connect marks 1 -> 0
Changed lines of the file:
@@
 $Descr A4 11693 8268
 encoding utf-8
-Sheet 1 5
+Sheet 1 1
 Title ""
 Date ""
@@
 	1    0    0    -1
 $EndComp
-NoConn ~ 8610 2980
 Wire Wire Line
 	8290 3390 9010 3390
@@
 Text Label 3670 2900 0    50   ~ 0
 PROGRAMMINGLED2
+Text Label 3670 1500 0    50   ~ 0
+SCLK
+$Comp
+L formula:HLMP-Q150-F0011 D?
+U 1 1 601FF02D
+P 3600 6800
+F 0 "D?" H 3593 7016 50  0000 C CNN
+F 1 "HLMP-Q150-F0011" H 3593 6925 50  0000 C CNN
+F 2 "footprints:HLMP-Q150-F0011" H 3500 6800 50  0001 C CNN
+F 3 "https://docs.broadcom.com/doc/AV02-3609EN" H 3600 6900 50  0001 C CNN
+F 4 "DK" H 3600 6800 60  0001 C CNN "MFN"
+F 5 "475-1410-1-ND" H 3600 6800 60  0001 C CNN "MPN"
+F 6 "https://www.digikey.com/products/en?keywords=475-1410-1-ND" H 4000 7300 60  0001 C CNN "PurchasingLink"
+	1    3600 6800
+	-1   0    0    1
+$EndComp
+$Comp
+L formula:HLMP-Q150-F0011 D?
+U 1 1 60200963
+P 3570 6410
+F 0 "D?" H 3563 6626 50  0000 C CNN
+F 1 "HLMP-Q150-F0011" H 3563 6535 50  0000 C CNN
+F 2 "footprints:HLMP-Q150-F0011" H 3470 6410 50  0001 C CNN
+F 3 "https://docs.broadcom.com/doc/AV02-3609EN" H 3570 6510 50  0001 C CNN
+F 4 "DK" H 3570 6410 60  0001 C CNN "MFN"
+F 5 "475-1410-1-ND" H 3570 6410 60  0001 C CNN "MPN"
+F 6 "https://www.digikey.com/products/en?keywords=475-1410-1-ND" H 3970 6910 60  0001 C CNN "PurchasingLink"
+	1    3570 6410
+	-1   0    0    1
+$EndComp
+Text Label 3670 3300 0    50   ~ 0
+DEBUG_LED1
+Text Label 3670 3400 0    50   ~ 0
+DEBUG_LED2
+Wire Wire Line
+	2720 6410 2420 6410
+Wire Wire Line
+	2730 6800 2430 6800
+Text Label 2420 6410 2    50   ~ 0
+DEBUG_LED1
+Text Label 2430 6800 2    50   ~ 0
+DEBUG_LED2
+Wire Wire Line
+	3020 6410 3420 6410
+Wire Wire Line
+	3030 6800 3450 6800
+$Comp
+L power:GND #PWR?
+U 1 1 602010BB
+P 4000 6410
+F 0 "#PWR?" H 4000 6160 50  0001 C CNN
+F 1 "GND" H 4005 6237 50  0000 C CNN
+F 2 "" H 4000 6410 50  0001 C CNN
+F 3 "" H 4000 6410 50  0001 C CNN
+	1    4000 6410
+	1    0    0    -1
+$EndComp
+$Comp
+L power:GND #PWR?
+U 1 1 602010C2
+P 4010 6800
+F 0 "#PWR?" H 4010 6550 50  0001 C CNN
+F 1 "GND" H 4015 6627 50  0000 C CNN
+F 2 "" H 4010 6800 50  0001 C CNN
+F 3 "" H 4010 6800 50  0001 C CNN
+	1    4010 6800
+	1    0    0    -1
+$EndComp
+Wire Wire Line
+	4010 6800 3750 6800
+Wire Wire Line
+	3720 6410 4000 6410
+$Comp
+L formula:R_3.01K R?
+U 1 1 6020AA87
+P 2870 6410
+F 0 "R?" V 2663 6410 50  0000 C CNN
+F 1 "R_3.01K" V 2754 6410 50  0000 C CNN
+F 2 "footprints:R_0805_OEM" H 2800 6410 50  0001 C CNN
+F 3 "http://www.yageo.com.tw/exep/pages/download/literatures/PYu-R_INT-thick_7.pdf" H 2950 6410 50  0001 C CNN
+F 4 "DK" H 2870 6410 60  0001 C CNN "MFN"
+F 5 "311-3.01KCRCT-ND" H 2870 6410 60  0001 C CNN "MPN"
+F 6 "https://www.digikey.com/products/en?keywords=311-3.01KCRCT-ND" H 3350 6810 60  0001 C CNN "PurchasingLink"
+	1    2870 6410
+	0    1    1    0
+$EndComp
+$Comp
+L formula:R_3.01K R?
+U 1 1 6020BAE1
+P 2880 6800
+F 0 "R?" V 2673 6800 50  0000 C CNN
+F 1 "R_3.01K" V 2764 6800 50  0000 C CNN
+F 2 "footprints:R_0805_OEM" H 2810 6800 50  0001 C CNN
+F 3 "http://www.yageo.com.tw/exep/pages/download/literatures/PYu-R_INT-thick_7.pdf" H 2960 6800 50  0001 C CNN
+F 4 "DK" H 2880 6800 60  0001 C CNN "MFN"
+F 5 "311-3.01KCRCT-ND" H 2880 6800 60  0001 C CNN "MPN"
+F 6 "https://www.digikey.com/products/en?keywords=311-3.01KCRCT-ND" H 3360 7200 60  0001 C CNN "PurchasingLink"
+	1    2880 6800
+	0    1    1    0
+$EndComp
 $EndSCHEMATC

Commit message: add debug leds
Other:
- note added: "DEBUG LEDS\n\n"
- note added: "PROGRAMMING LEDS\n\n"
- moved on the sheet: D?, R?

Commit message: Edit schematics
Parts:
- removed C?: C_0.1uF, footprints:C_0805_OEM, symbol formula:C_0.1uF
- removed DS?: AMC1602AR-B-Y6WFDY-SPI, Display:HY1602E, symbol formula:AMC1602AR-B-Y6WFDY-SPI
- removed R?: R_1.13K, footprints:R_0805_OEM, symbol formula:R_1.13K
- removed R?: R_4.99K, footprints:R_0805_OEM, symbol formula:R_4.99K
- added C?: C_0.1uF, footprints:C_0805_OEM, symbol formula:C_0.1uF
- added C?: C_100pF, footprints:C_0805_OEM, symbol formula:C_100pF
- added J? (x2): UF_4_VT, footprints:Ultrafit_4, symbol formula:UF_4_VT
- added J? (x2): UF_5_VT, symbol formula:UF_5_VT
- added R?: R_100, footprints:R_0805_OEM, symbol formula:R_100
- added R? (x4): R_4.7K, footprints:R_0805_OEM, symbol formula:R_4.7K
- added U? (x2): COM-11441, Display_7Segment:CA56-12EWA, symbol formula:COM-11441
Connections:
- net labels added: CS_I, CS_V, CURRENT_MONITOR, FA_DO_SIGNALS, FLYBACK_CHARGE, SDI, SS, SS_I, SS_V, VOLTAGE_MONITOR
- net labels removed: CS, CSB, RS, SCLK, SID
- wire segments 59 -> 75
- no-connect marks 0 -> 14
Other:
- note added: "7 SEGMENT DISPLAY FOR CURRENT\n"
- note added: "7 SEGMENT DISPLAY FOR VOLTAGE\n"
- note added: "ATMEGA16M1 PROGRAMMING HEADER"
- note added: "CONNECTOR FOR 7 SEGMENT DISPLAY CURRENT"
- note added: "CONNECTOR FOR 7 SEGMENT DISPLAY VOLTAGE"
- note added: "CONNECTOR FOR CURRENT KNOB"
- note added: "CONNECTOR FOR VOLTAGE KNOB"
- note removed: "LCD DISPLAY\n"
- moved on the sheet: J?, R?, SW1?, SW?

Commit message: edit schematics
Connections:
- net labels added: DCDC_CONVERTER, DONE_SIGNAL, FAULT_SIGNAL
- net labels removed: FA_DO_SIGNALS, SS
- no-connect marks 14 -> 12
Changed lines of the file:
@@
 $EndComp
 $Comp
-L power:GND #PWR?
+L power:GND #PWR0101
 U 1 1 5FA510AE
 P 4220 4820
-F 0 "#PWR?" H 4220 4570 50  0001 C CNN
+F 0 "#PWR0101" H 4220 4570 50  0001 C CNN
 F 1 "GND" H 4225 4647 50  0000 C CNN
 F 2 "" H 4220 4820 50  0001 C CNN
@@
 $EndComp
 $Comp
-L power:GND #PWR?
+L power:GND #PWR0102
 U 1 1 5FA51C2A
 P 4790 4820
-F 0 "#PWR?" H 4790 4570 50  0001 C CNN
+F 0 "#PWR0102" H 4790 4570 50  0001 C CNN
 F 1 "GND" H 4795 4647 50  0000 C CNN
 F 2 "" H 4790 4820 50  0001 C CNN
@@
 $EndComp
 $Comp
-L power:GND #PWR?
+L power:GND #PWR0103
 U 1 1 5FA522F4
 P 4520 4700
-F 0 "#PWR?" H 4520 4450 50  0001 C CNN
+F 0 "#PWR0103" H 4520 4450 50  0001 C CNN
 F 1 "GND" H 4525 4527 50  0000 C CNN
 F 2 "" H 4520 4700 50  0001 C CNN
@@
 	4790 4480 4790 4520
 $Comp
-L power:GND #PWR?
+L power:GND #PWR0104
 U 1 1 5FA55995
 P 4920 4170
-F 0 "#PWR?" H 4920 3920 50  0001 C CNN
+F 0 "#PWR0104" H 4920 3920 50  0001 C CNN
 F 1 "GND" H 4925 3997 50  0000 C CNN
 F 2 "" H 4920 4170 50  0001 C CNN
@@
 MOSI
 $Comp
-L power:VCC #PWR?
+L power:VCC #PWR0105
 U 1 1 5FA62F57
 P 5990 6980
-F 0 "#PWR?" H 5990 6830 50  0001 C CNN
+F 0 "#PWR0105" H 5990 6830 50  0001 C CNN
 F 1 "VCC" H 6005 7153 50  0000 C CNN
 F 2 "" H 5990 6980 50  0001 C CNN
@@
 $EndComp
 $Comp
-L power:GND #PWR?
+L power:GND #PWR0106
 U 1 1 5FA63844
 P 5990 7180
-F 0 "#PWR?" H 5990 6930 50  0001 C CNN
+F 0 "#PWR0106" H 5990 6930 50  0001 C CNN
 F 1 "GND" H 5995 7007 50  0000 C CNN
 F 2 "" H 5990 7180 50  0001 C CNN
@@
 	2980 5680 2680 5680
 $Comp
-L power:GND #PWR?
+L power:GND #PWR0107
 U 1 1 5FA6AC79
 P 4150 5680
-F 0 "#PWR?" H 4150 5430 50  0001 C CNN
+F 0 "#PWR0107" H 4150 5430 50  0001 C CNN
 F 1 "GND" H 4155 5507 50  0000 C CNN
 F 2 "" H 4150 5680 50  0001 C CNN
@@
 	2990 6070 2690 6070
 $Comp
-L power:GND #PWR?
+L power:GND #PWR0108
 U 1 1 5FA6CB5F
 P 4160 6070
-F 0 "#PWR?" H 4160 5820 50  0001 C CNN
+F 0 "#PWR0108" H 4160 5820 50  0001 C CNN
 F 1 "GND" H 4165 5897 50  0000 C CNN
 F 2 "" H 4160 6070 50  0001 C CNN
@@
 PROGRAMMINGLED2
 $Comp
-L power:VCC #PWR?
+L power:VCC #PWR0109
 U 1 1 5FA6F6D3
 P 10460 5020
-F 0 "#PWR?" H 10460 4870 50  0001 C CNN
+F 0 "#PWR0109" H 10460 4870 50  0001 C CNN
 F 1 "VCC" H 10475 5193 50  0000 C CNN
 F 2 "" H 10460 5020 50  0001 C CNN
@@
 $EndComp
 $Comp
-L power:GND #PWR?
+L power:GND #PWR0110
 U 1 1 5FA70E3A
 P 10460 5170
-F 0 "#PWR?" H 10460 4920 50  0001 C CNN
+F 0 "#PWR0110" H 10460 4920 50  0001 C CNN
 F 1 "GND" H 10465 4997 50  0000 C CNN
 F 2 "" H 10460 5170 50  0001 C CNN
@@
 CS_V
 $Comp
-L power:GND #PWR?
+L power:GND #PWR0111
 U 1 1 5FA570DD
 P 9230 4970
-F 0 "#PWR?" H 9230 4720 50  0001 C CNN
+F 0 "#PWR0111" H 9230 4720 50  0001 C CNN
 F 1 "GND" H 9235 4797 50  0000 C CNN
 F 2 "" H 9230 4970 50  0001 C CNN
@@
 $EndComp
 $Comp
-L power:VCC #PWR?
+L power:VCC #PWR0112
 U 1 1 5FA6194E
 P 10480 5960
-F 0 "#PWR?" H 10480 5810 50  0001 C CNN
+F 0 "#PWR0112" H 10480 5810 50  0001 C CNN
 F 1 "VCC" H 10495 6133 50  0000 C CNN
 F 2 "" H 10480 5960 50  0001 C CNN
@@
 $EndComp
 $Comp
-L power:GND #PWR?
+L power:GND #PWR0113
 U 1 1 5FA61954
 P 10480 6110
-F 0 "#PWR?" H 10480 5860 50  0001 C CNN
+F 0 "#PWR0113" H 10480 5860 50  0001 C CNN
 F 1 "GND" H 10485 5937 50  0000 C CNN
 F 2 "" H 10480 6110 50  0001 C CNN
@@
 CS_I
 $Comp
-L power:GND #PWR?
+L power:GND #PWR0114
 U 1 1 5FA6195F
 P 9250 5910
-F 0 "#PWR?" H 9250 5660 50  0001 C CNN
+F 0 "#PWR0114" H 9250 5660 50  0001 C CNN
 F 1 "GND" H 9255 5737 50  0000 C CNN
 F 2 "" H 9250 5910 50  0001 C CNN
@@
 	5060 3750 5060 3850
 $Comp
-L power:VCC #PWR?
+L power:VCC #PWR0115
 U 1 1 5FA56CA3
 P 5060 3750
-F 0 "#PWR?" H 5060 3600 50  0001 C CNN
+F 0 "#PWR0115" H 5060 3600 50  0001 C CNN
 F 1 "VCC" H 5075 3923 50  0000 C CNN
 F 2 "" H 5060 3750 50  0001 C CNN
@@
 	3190 7140 3610 7140
 $Comp
-L power:GND #PWR?
+L power:GND #PWR0116
 U 1 1 602010BB
 P 4160 6750
-F 0 "#PWR?" H 4160 6500 50  0001 C CNN
+F 0 "#PWR0116" H 4160 6500 50  0001 C CNN
 F 1 "GND" H 4165 6577 50  0000 C CNN
 F 2 "" H 4160 6750 50  0001 C CNN
@@
 $EndComp
 $Comp
-L power:GND #PWR?
+L power:GND #PWR0117
 U 1 1 602010C2
 P 4170 7140
-F 0 "#PWR?" H 4170 6890 50  0001 C CNN
+F 0 "#PWR0117" H 4170 6890 50  0001 C CNN
 F 1 "GND" H 4175 6967 50  0000 C CNN
 F 2 "" H 4170 7140 50  0001 C CNN
@@
 NoConn ~ 1470 2200
 $Comp
-L power:VCC #PWR?
+L power:VCC #PWR0118
 U 1 1 60277D9C
 P 890 1400
-F 0 "#PWR?" H 890 1250 50  0001 C CNN
+F 0 "#PWR0118" H 890 1250 50  0001 C CNN
 F 1 "VCC" H 905 1573 50  0000 C CNN
 F 2 "" H 890 1400 50  0001 C CNN
@@
 Connection ~ 1360 1800
 $Comp
-L power:GND #PWR?
+L power:GND #PWR0119
 U 1 1 60282627
 P 1360 2270
-F 0 "#PWR?" H 1360 2020 50  0001 C CNN
+F 0 "#PWR0119" H 1360 2020 50  0001 C CNN
 F 1 "GND" H 1365 2097 50  0000 C CNN
 F 2 "" H 1360 2270 50  0001 C CNN
@@
 	1360 2150 1360 2270
 $Comp
-L power:GND #PWR?
+L power:GND #PWR0120
 U 1 1 60285595
 P 890 1950
-F 0 "#PWR?" H 890 1700 50  0001 C CNN
+F 0 "#PWR0120" H 890 1700 50  0001 C CNN
 F 1 "GND" H 895 1777 50  0000 C CNN
 F 2 "" H 890 1950 50  0001 C CNN
@@
 	890  1880 890  1950
 $Comp
-L power:GND #PWR?
+L power:GND #PWR0121
 U 1 1 60288BAA
 P 1350 4480
-F 0 "#PWR?" H 1350 4230 50  0001 C CNN
+F 0 "#PWR0121" H 1350 4230 50  0001 C CNN
 F 1 "GND" H 1355 4307 50  0000 C CNN
 F 2 "" H 1350 4480 50  0001 C CNN
@@
 ATMEGA16M1 PROGRAMMING HEADER
 Text Label 3670 2500 0    50   ~ 0
-FA_DO_SIGNALS
+FAULT_SIGNAL
 Text Label 3670 3000 0    50   ~ 0
 FLYBACK_CHARGE
@@
 Wire Wire Line
 	4400 3970 4400 4200
-NoConn ~ 3670 2600
-NoConn ~ 3670 2700
 $Comp
 L formula:COM-11441 U?
@@
 $EndComp
 $Comp
-L power:VCC #PWR?
+L power:VCC #PWR0122
 U 1 1 603B43F7
 P 8140 2070
-F 0 "#PWR?" H 8140 1920 50  0001 C CNN
+F 0 "#PWR0122" H 8140 1920 50  0001 C CNN
 F 1 "VCC" H 8155 2243 50  0000 C CNN
 F 2 "" H 8140 2070 50  0001 C CNN
@@
 	8140 2070 8530 2070
 $Comp
-L power:GND #PWR?
+L power:GND #PWR0123
 U 1 1 603ADD9F
 P 8430 2170
-F 0 "#PWR?" H 8430 1920 50  0001 C CNN
+F 0 "#PWR0123" H 8430 1920 50  0001 C CNN
 F 1 "GND" H 8435 1997 50  0000 C CNN
 F 2 "" H 8430 2170 50  0001 C CNN
@@
 	8530 2170 8430 2170
 Text Label 8530 1570 2    50   ~ 0
-SS
+SS_V
 Text Label 8530 1670 2    50   ~ 0
 SDI
@@
 SCK
 $Comp
-L power:VCC #PWR?
+L power:VCC #PWR0124
 U 1 1 603DA40F
 P 6540 4400
-F 0 "#PWR?" H 6540 4250 50  0001 C CNN
+F 0 "#PWR0124" H 6540 4250 50  0001 C CNN
 F 1 "VCC" H 6555 4573 50  0000 C CNN
 F 2 "" H 6540 4400 50  0001 C CNN
@@
 	6540 4400 6800 4400
 $Comp
-L power:GND #PWR?
+L power:GND #PWR0125
 U 1 1 603DE9CA
 P 6900 4380
-F 0 "#PWR?" H 6900 4130 50  0001 C CNN
+F 0 "#PWR0125" H 6900 4130 50  0001 C CNN
 F 1 "GND" H 6905 4207 50  0000 C CNN
 F 2 "" H 6900 4380 50  0001 C CNN
@@
 $EndComp
 $Comp
-L power:GND #PWR?
+L power:GND #PWR0126
 U 1 1 603DFA87
 P 6670 2440
-F 0 "#PWR?" H 6670 2190 50  0001 C CNN
+F 0 "#PWR0126" H 6670 2190 50  0001 C CNN
 F 1 "GND" H 6675 2267 50  0000 C CNN
 F 2 "" H 6670 2440 50  0001 C CNN
@@
 	6800 2440 6800 2670
 $Comp
-L power:GND #PWR?
+L power:GND #PWR0127
 U 1 1 603E5BBD
 P 6620 1240
-F 0 "#PWR?" H 6620 990 50  0001 C CNN
+F 0 "#PWR0127" H 6620 990 50  0001 C CNN
 F 1 "GND" H 6625 1067 50  0000 C CNN
 F 2 "" H 6620 1240 50  0001 C CNN
@@
 	6130 1530 5920 1530
 $Comp
-L power:VCC #PWR?
+L power:VCC #PWR0128
 U 1 1 603F1FCE
 P 6130 1170
-F 0 "#PWR?" H 6130 1020 50  0001 C CNN
+F 0 "#PWR0128" H 6130 1020 50  0001 C CNN
 F 1 "VCC" H 6145 1343 50  0000 C CNN
 F 2 "" H 6130 1170 50  0001 C CNN
@@
 $EndComp
 $Comp
-L power:VCC #PWR?
+L power:VCC #PWR0129
 U 1 1 603F8D80
 P 6240 2410
-F 0 "#PWR?" H 6240 2260 50  0001 C CNN
+F 0 "#PWR0129" H 6240 2260 50  0001 C CNN
 F 1 "VCC" H 6255 2583 50  0000 C CNN
 F 2 "" H 6240 2410 50  0001 C CNN
@@
 $EndComp
 $Comp
-L power:VCC #PWR?
+L power:VCC #PWR0130
 U 1 1 604024E5
 P 6370 3620
-F 0 "#PWR?" H 6370 3470 50  0001 C CNN
+F 0 "#PWR0130" H 6370 3470 50  0001 C CNN
 F 1 "VCC" H 6385 3793 50  0000 C CNN
 F 2 "" H 6370 3620 50  0001 C CNN
@@
 $EndComp
 $Comp
-L power:VCC #PWR?
+L power:VCC #PWR0131
 U 1 1 603E739B
 P 8130 3810
-F 0 "#PWR?" H 8130 3660 50  0001 C CNN
+F 0 "#PWR0131" H 8130 3660 50  0001 C CNN
 F 1 "VCC" H 8145 3983 50  0000 C CNN
 F 2 "" H 8130 3810 50  0001 C CNN
@@
 	8130 3810 8520 3810
 $Comp
-L power:GND #PWR?
+L power:GND #PWR0132
 U 1 1 603E73A2
 P 8420 3910
-F 0 "#PWR?" H 8420 3660 50  0001 C CNN
+F 0 "#PWR0132" H 8420 3660 50  0001 C CNN
 F 1 "GND" H 8425 3737 50  0000 C CNN
 F 2 "" H 8420 3910 50  0001 C CNN
@@
 	8520 3910 8420 3910
 Text Label 8520 3310 2    50   ~ 0
-SS
+SS_I
 Text Label 8520 3410 2    50   ~ 0
 SDI
@@
 SCK
 $Comp
-L power:VCC #PWR?
+L power:VCC #PWR0133
 U 1 1 603EDB7A
 P 6390 5960
-F 0 "#PWR?" H 6390 5810 50  0001 C CNN
+F 0 "#PWR0133" H 6390 5810 50  0001 C CNN
 F 1 "VCC" H 6405 6133 50  0000 C CNN
 F 2 "" H 6390 5960 50  0001 C CNN
@@
 	6390 5960 6650 5960
 $Comp
-L power:GND #PWR?
+L power:GND #PWR0134
 U 1 1 603EDB81
 P 6750 5940
-F 0 "#PWR?" H 6750 5690 50  0001 C CNN
+F 0 "#PWR0134" H 6750 5690 50  0001 C CNN
 F 1 "GND" H 6755 5767 50  0000 C CNN
 F 2 "" H 6750 5940 50  0001 C CNN
@@
 $EndComp
 $Comp
-L power:VCC #PWR?
+L power:VCC #PWR0135
 U 1 1 603EDB92
 P 6220 5180
-F 0 "#PWR?" H 6220 5030 50  0001 C CNN
+F 0 "#PWR0135" H 6220 5030 50  0001 C CNN
 F 1 "VCC" H 6235 5353 50  0000 C CNN
 F 2 "" H 6220 5180 50  0001 C CNN
@@
 Text Label 5830 5540 2    50   ~ 0
 SS_I
+Text Label 3670 2400 0    50   ~ 0
+SS_V
+Text Label 3670 1500 0    50   ~ 0
+SS_I
+Text Label 3670 2600 0    50   ~ 0
+DONE_SIGNAL
+Text Label 3670 2700 0    50   ~ 0
+DCDC_CONVERTER
 $EndSCHEMATC

Commit message: edit schematics
Parts:
- removed D? (x2): HLMP-Q150-F0011, footprints:HLMP-Q150-F0011, symbol formula:HLMP-Q150-F0011
- removed R? (x2): R_3.01K, footprints:R_0805_OEM, symbol formula:R_3.01K
- added D? (x2): 12B-x, footprints:HLMP-Q150-F0011, symbol formula:12B-x
- added R? (x2): R_1.13K, footprints:R_0805_OEM, symbol formula:R_1.13K
- added R? (x2): R_3.01K, footprints:R_0805_OEM, symbol formula:R_3.01K
- added U? (x2): TLP175A_OEM, footprints:MFSOP6-4_4.4x3.6mm_Pitch1.27mm_OEM, symbol formula:TLP175A_OEM
Connections:
- net labels added: 12V
- wire segments 75 -> 86
Other:
- moved on the sheet: D?, R?

Commit message: edit schematics
Parts:
- removed D? (x2): 12B-x, footprints:HLMP-Q150-F0011, symbol formula:12B-x
- removed J? (x2): UF_4_VT, footprints:Ultrafit_4, symbol formula:UF_4_VT
- removed R? (x2): R_4.7K, footprints:R_0805_OEM, symbol formula:R_4.7K
- removed R? (x2): R_1.13K, footprints:R_0805_OEM, symbol formula:R_1.13K
- removed R? (x2): R_3.01K, footprints:R_0805_OEM, symbol formula:R_3.01K
- removed U? (x2): TLP175A_OEM, footprints:MFSOP6-4_4.4x3.6mm_Pitch1.27mm_OEM, symbol formula:TLP175A_OEM
- added D? (x2): Q8P7BXXG02E, footprints:LED_0805_OEM, symbol formula:Q8P7BXXG02E
- added J?: UF_5_VT, symbol formula:UF_5_VT
- added J?: CONN_01x04, Pin_Headers:Pin_Header_Straight_1x04_Pitch2.54mm, symbol formula:CONN_01x04
- added R?: R_4.7K, footprints:R_0805_OEM, symbol formula:R_4.7K
- added R? (x2): R_200, footprints:R_0805_OEM, symbol formula:R_200
Connections:
- net labels added: 1, 2, 3, 4, CS
- net labels removed: 12V, CS_I, CS_V, D_OUTPUT_I
- wire segments 86 -> 80
- no-connect marks 12 -> 14
Other:
- note added: "CONNECTOR FOR ROTARY ENCODERS"
- note removed: "CONNECTOR FOR CURRENT KNOB"
- note removed: "CONNECTOR FOR VOLTAGE KNOB"
- moved on the sheet: SW1?, SW?
