File: hv_power_supply/power_supply/flyback_converter.sch (KiCad schematic (older format))
At the start: 0 parts

Commit message: Started importing flyback schematic, still quite a few passives that I need to make
Parts:
- added C?: C_2.2uF, footprints:C_0805_OEM, symbol formula:C_2.2uF
- added C? (x4): C, footprints:C_0805_OEM, symbol formula:C_2.2uF
- added C?: C_10uF_450V, footprints:C_10uF_450V, symbol formula:C_10uF_450V
- added D?: RFN5TF8S, formula:TO-220NFM, symbol formula:RFN5TF8S
- added Q?: NTB35N15, formula:D2PAK, symbol formula:NTB35N15
- added R? (x2): R_100K, footprints:R_0805_OEM, symbol formula:R_100K
- added R?: R_0, footprints:R_0603_1608Metric, symbol formula:R_0
- added T?: GA3460-BL, formula:GA3460-BL, symbol formula:GA3460-BL
- added U?: LT3751, formula:TSSOP-20_EXPOSED_PAD, symbol formula:LT3751
- added U?: ACPL-C87B-000E, formula:SSO-8, symbol formula:ACPL-C87B-000E
Connections:
- net labels added: +24V, GND, GNDPWR, HV_OUT, VCC
- wire segments 0 -> 28
Other:
- note added: "5x2.2uF"
