File: hv_power_supply/power_supply/flyback_converter.sch (KiCad schematic (older format))
At the start: 14 parts

Commit message: First pass at full flyback schematic... Still working on some auxilary circuitry
Parts:
- removed Q?: NTB35N15, formula:D2PAK, symbol formula:NTB35N15
- removed R?: R_0, footprints:R_0603_1608Metric, symbol formula:R_0
- removed T?: GA3460-BL, formula:GA3460-BL, symbol formula:GA3460-BL
- removed U?: LT3751, formula:TSSOP-20_EXPOSED_PAD, symbol formula:LT3751
- added C?: C_10uF_50V, footprints:C_0805_OEM, symbol formula:C_10uF_50V
- added C? (x2): C_100nF, footprints:C_0603_1608Metric, symbol formula:C_100nF
- added C?: C_10nF, footprints:C_0805_OEM, symbol formula:C_10nF
- added C?: C_0.47uF, formula:1812(4532Metric), symbol formula:C_0.47uF_450V
- added C? (x4): C_0.1uF, footprints:C_0805_OEM, symbol formula:C_0.1uF
- added C?: C_10uF, footprints:C_0805_OEM, symbol formula:C_10uF_16V
- added C?: C_10uF_16V, footprints:C_0805_OEM, symbol formula:C_10uF_16V
- added C? (x2): C_100pF, footprints:C_0805_OEM, symbol formula:C_100pF
- added Q?: FDB33N25, formula:D2PAK, symbol formula:FDB33N25
- added R?: R_6mOhm, formula:R_2512_LARGE, symbol formula:R_6mOhm
- added R? (x2): R_200K, footprints:R_0805_OEM, symbol formula:R_200K
- added R? (x2): R_576K, footprints:R_0805_OEM, symbol formula:R_576K
- added R?: R_80.6k, footprints:R_0805_OEM, symbol formula:R_80.6k
- added R?: R_36.5k, footprints:R_0805_OEM, symbol formula:R_36.5k
- added R?: R_536k, formula:R_2010_Vishay, symbol formula:R_536k
- added R?: R_1.5k, formula:R_2010_Vishay, symbol formula:R_1.5k
- added R?: R_100K, footprints:R_0805_OEM, symbol formula:R_100K
- added R? (x4): R_10K, footprints:R_0805_OEM, symbol formula:R_10K
- added R?: DNP, footprints:R_0603_1608Metric, symbol formula:R_0
- added T?: GA3460-BL, formula:GA3460-BL, symbol formula:GA3460-BL
- added U?: LT3751, formula:TSSOP-20_EXPOSED_PAD, symbol formula:LT3751
- added U?: LT-1997-2, formula:16(12)-MSOP, symbol formula:LT-1997-2
- added U?: AD623, symbol formula:AD623
- C?: value C_10uF_450V -> C_10uF
Connections:
- net labels added: +5V, -5V, FB_SIGNAL, HV_5V, MCU_CHARGE, MCU_DAC(.6-4.4), MCU_DONE, MCU_FAULT, MCU_OFFSET_SHDN, V_FB+, V_FB-
- net labels removed: VCC
- wire segments 28 -> 179
- no-connect marks 0 -> 2
Other:
- note added: "GAIN: .125\nDATASHEET pg 16"
- moved on the sheet: C?, D?, R?, U?

Commit message: added RCD clamp and 2nd order RC snubber
Parts:
- removed T?: GA3460-BL, formula:GA3460-BL, symbol formula:GA3460-BL
- added C17, C18: C_10nF, footprints:C_0805_OEM, symbol formula:C_10nF
- added C6: C_1uF, footprints:C_0805_OEM, symbol formula:C_1uF
- added D1: 1N5369B, footprints:DO-214AA, symbol formula:D_Zener_18V
- added R14: R_1K, footprints:R_0805_OEM, symbol formula:R_1K
- added R17, R18: R_10, footprints:R_2512_OEM, symbol formula:R_13_2W_2512_0
- added T1: GA3460-BL, footprints:GA3460-BL, symbol formula:GA3460-BL
- gave numbers to parts that had none: 42
Connections:
- wire segments 179 -> 201

Commit message: make schematic sheets talk to each other
Parts:
- removed C1, C10, C2, C8: C_0.1uF, footprints:C_0805_OEM, symbol formula:C_0.1uF
- removed C12: C_10uF, footprints:C_0805_OEM, symbol formula:C_10uF_16V
- removed C16, C19: C_100nF, footprints:C_0603_1608Metric, symbol formula:C_100nF
- removed C17, C18: C_10nF, footprints:C_0805_OEM, symbol formula:C_10nF
- removed C20: C_0.47uF, formula:1812(4532Metric), symbol formula:C_0.47uF_450V
- removed C21: C_10uF, footprints:C_10uF_450V, symbol formula:C_10uF_450V
- removed C3, C4: C_100pF, footprints:C_0805_OEM, symbol formula:C_100pF
- removed C7: C_10uF_16V, footprints:C_0805_OEM, symbol formula:C_10uF_16V
- removed D1: 1N5369B, footprints:DO-214AA, symbol formula:D_Zener_18V
- removed R1: R_100K, footprints:R_0805_OEM, symbol formula:R_100K
- removed R10, R11, R2, R3: R_10K, footprints:R_0805_OEM, symbol formula:R_10K
- removed R13: DNP, footprints:R_0603_1608Metric, symbol formula:R_0
- removed R14: R_1K, footprints:R_0805_OEM, symbol formula:R_1K
- removed R17, R18: R_10, footprints:R_2512_OEM, symbol formula:R_13_2W_2512_0
- removed R19: R_536k, formula:R_2010_Vishay, symbol formula:R_536k
- removed U1: LT-1997-2, formula:16(12)-MSOP, symbol formula:LT-1997-2
- removed U3: AD623, symbol formula:AD623
- removed U4: ACPL-C87B-000E, formula:SSO-8, symbol formula:ACPL-C87B-000E
- added C10: C_0.47uF, footprints:1812(4532Metric), symbol formula:C_0.47uF_450V
- added C11, C12, C13: C_10uF, footprints:C_10uF_450V, symbol formula:C_10uF_450V
- added C8, C9: C_4.7nF, footprints:C_1206_OEM, symbol formula:C_4.7nF
- added D1: FSF10A20, formula:TO-220NFM, symbol formula:FSF10A20
- added R11, R12: R_13, formula:R_2512_LARGE, symbol formula:R_13_2W_2512_0
- added R13, R14, R15, R16, R17, R18, R19, R20: R_67k, footprints:R_0805_OEM, symbol formula:R_67k
- added R8: R_1K, footprints:R_2512_OEM, symbol formula:R_1K_HV
- renumbered C5 to C1, C22 to C14, C6 to C2, C9 to C3, C11 to C4, C13 to C5, C14 to C6, C15 to C7, R4 to R1, R16 to R10, R5 to R2, R20 to R21, R6 to R3, R7 to R4, R8 to R5, R9 to R6, R12 to R7, R15 to R9, U2 to U1
Connections:
- net labels added: CHARGE, HV+, HV-, HV_V_FB, LV_V_FB, ~DONE, ~FAULT
- net labels removed: -5V, FB_SIGNAL, GNDPWR, HV_5V, HV_OUT, MCU_CHARGE, MCU_DAC(.6-4.4), MCU_DONE, MCU_FAULT, MCU_OFFSET_SHDN, V_FB+, V_FB-
- wire segments 201 -> 129
Other:
- note removed: "GAIN: .125\nDATASHEET pg 16"
- moved on the sheet: C1, C14, C2, C3, C4, C5, C6, C7, D2, Q1, R1, R10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
