File: hv_power_supply/power_supply/power_supply.kicad_pcb (KiCad board)
At the start: 4 copper layers, 123 parts, among them J1 CONN_01x04, J2 CONN_02X03, J3 UF_5_VT, J4 UF_5_VT, J5 UF_5_VT, J6 CONN_01x02, J7 MegaFit_06_RA, J8 MegaFit_06_RA, K1 CPC1979J, Q1 FDB33N25, Q2 SSM3K333R, Q3 SSM3K333R, Q4 FQD2N60CTM, T1 GA3460-BL, U1 LT3751, U10 LT-1997-2, U11 ADA4661-2, U2 MAXM15464, U3 ATMEGA16M1, U6 LTC1983ES6-5#TRMPBF, U7 CPC1117NTR, U8 ACPL-C79B-500E, U9 ACPL-C87B-000E, Y1 Crystal_SMD

Commit message: Most of placement done, beginning routing.
Parts:
- moved J7 249.6 mm to (186.7, 160.0)
- moved R40 240.0 mm to (24.1, 69.8), turned to 90 degrees
- moved Q4 235.5 mm to (41.9, 94.0), turned to 90 degrees
- moved R38 232.4 mm to (27.9, 116.8)
- moved U8 215.3 mm to (100.3, 90.2), turned to 270 degrees
- moved C27 210.9 mm to (90.2, 87.6), turned to 180 degrees
- moved C26 205.6 mm to (27.9, 71.1), turned to 180 degrees
- moved R37 204.3 mm to (31.8, 69.8), turned to 90 degrees
- moved R44 203.5 mm to (143.5, 114.3), turned to 90 degrees
- moved U9 202.5 mm to (100.3, 102.9), turned to 270 degrees
- moved U10 200.0 mm to (134.6, 105.4), turned to 270 degrees
- moved C24 198.4 mm to (90.2, 83.8), turned to 180 degrees
- moved R47 198.0 mm to (153.7, 108.0)
- moved PS1 198.0 mm to (100.3, 77.5), turned to 180 degrees
- moved C22 197.9 mm to (110.5, 100.3)
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Connections:
- K1 pad 1: /Flyback Converter/HV+ -> Net-(F1-Pad1)
- K1 pad 2: Net-(F1-Pad1) -> /Flyback Converter/HV+
- U8 pad 1: +5V -> /Protections/HV_5V
- U8 pad 2: /Protections/I_LV+ -> Net-(C26-Pad1)
- U8 pad 3: /Protections/I_LV- -> Net-(C26-Pad2)
- U8 pad 4: GND -> /Flyback Converter/HV-
- U8 pad 5: /Flyback Converter/HV- -> GND
- U8 pad 6: Net-(C26-Pad2) -> /Protections/I_LV-
- U8 pad 7: Net-(C26-Pad1) -> /Protections/I_LV+
- U8 pad 8: /Protections/HV_5V -> +5V
Other:
- board text added: "+5V"
- board text added: "-5V"

Commit message: All routing finished except for 5V and GND... Need to look into adding input filtering to power supply chips and some GND separation between LV, Flyback, and HV
Parts:
- moved R31 161.4 mm to (122.7, 55.6)
- moved J1 142.8 mm to (139.7, 74.9), turned to 90 degrees
- moved J2 141.5 mm to (133.3, 67.3), turned to 180 degrees
- moved R23 114.3 mm to (139.7, 71.1), turned to 270 degrees
- moved R24 106.2 mm to (144.8, 71.1), turned to 270 degrees
- moved R25 96.1 mm to (163.8, 54.6)
- moved R30 95.7 mm to (194.3, 72.4), turned to 90 degrees
- moved J4 95.6 mm to (141.0, 50.8), turned to 270 degrees
- moved J3 88.4 mm to (185.4, 64.8)
- moved J5 82.2 mm to (198.1, 64.8)
- moved R26 80.5 mm to (163.8, 52.1)
- moved R28 80.1 mm to (181.6, 72.4), turned to 90 degrees
- moved R27 79.3 mm to (137.2, 62.2), turned to 90 degrees
- moved R29 72.6 mm to (149.9, 45.7), turned to 270 degrees
- moved R6 71.6 mm to (164.5, 80.6)
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Connections:
- net Net-(C26-Pad1) renamed /Protections/I_HV+
- net Net-(C26-Pad2) renamed /Protections/I_HV-
- net Net-(C28-Pad2) renamed /Protections/V_FB_LV-
- net Net-(C29-Pad1) renamed /Protections/V_FB_LV+
- net Net-(C36-Pad2) renamed /Protections/I_LV_N
- net Net-(C37-Pad1) renamed /Protections/I_LV_P
- J2 pad 3: /User Interface/SCK -> /User Interface/SCK_PROG
- U3 pad 12: /User Interface/SCK -> /User Interface/SCK_PROG
Routing:
- net /Flyback Converter/LV_V_FB: track 0.00 -> 126.4 mm, vias 0 -> 2
- net /Flyback Converter/CHARGE: track 0.00 -> 118.7 mm, vias 0 -> 2
- net /Flyback Converter/~FAULT: track 0.00 -> 115.8 mm, vias 0 -> 2
- net /Flyback Converter/~DONE: track 0.00 -> 110.7 mm
- net Net-(Q4-Pad1): track 0.00 -> 78.9 mm, vias 0 -> 2
- net /Protections/I_HV-: track 0.00 -> 68.2 mm
- net /Protections/I_HV+: track 0.00 -> 67.6 mm
- net /-5V Buck Converter/~-5V_SHDN: track 0.00 -> 61.0 mm, vias 0 -> 2
- net /User Interface/SS_V: track 0.00 -> 56.7 mm, vias 0 -> 2
- net /Protections/I_LV_P: track 0.00 -> 56.0 mm
- net /Protections/I_LV_N: track 0.00 -> 54.7 mm
- net /Protections/~MCU_OFFSET_SHDN: track 0.00 -> 50.7 mm, vias 0 -> 2
- net /User Interface/SCK: track 0.00 -> 50.6 mm, vias 0 -> 1
- net /Protections/HV_5V_CTRL: track 0.00 -> 47.9 mm, vias 0 -> 2
- net /Protections/Out&nDis: track 0.00 -> 46.8 mm
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- added copper zone on In2.Cu, net +5V
- added copper zone on In2.Cu, net /-5V Buck Converter/-5V
- added copper zone on B.Cu, net /Buck Converter/+24V
- added copper zone on F.Cu, net /Buck Converter/+24V
- added copper zone on F.Cu, net /Flyback Converter/HV+
- added copper zone on In2.Cu, net /Flyback Converter/HV+
- added copper zone on F.Cu, net /Flyback Converter/HV-
- added copper zone on In1.Cu, net /Flyback Converter/HV-
- added copper zone on B.Cu, net /Protections/HV_5V
- added copper zone on F.Cu, net GND
- added copper zone on In1.Cu, net GND
- added copper zone on B.Cu, net Net-(C2-Pad2)
- added copper zone on F.Cu, net Net-(C2-Pad2)
- added copper zone on B.Cu, net Net-(C8-Pad1)
- added copper zone on F.Cu, net Net-(C8-Pad1)
- added copper zone on F.Cu, net Net-(D2-Pad1)
- added copper zone on B.Cu, net Net-(Q1-Pad3)
- added copper zone on F.Cu, net Net-(Q1-Pad3)
Other:
- board text removed: "+5V"
