File: hardware_in_the_loop/boards/hitl_system_interface/oem_HitLInterface_board/HitLSystemInterfaceSchematic/SystemHitLSInterface.sch (KiCad schematic (older format))
At the start: 44 parts, among them J1 CONN_02X03, J2 NanoFit_RA_SMT_08, U1 MCP2561-E_SN, U3 USB_MicroB, U4 FT232RL

Commit message: Finished Electrical Design Checklist
Parts:
- removed C1: C_0.1uF, footprints:C_0805_OEM, symbol template-rescue:C_0.1uF-formula
- removed J2: NanoFit_RA_SMT_08, footprints:NanoFit_RA_8, symbol formula:NanoFit_RA_SMT_08
- removed R2: R_200, footprints:R_0805_OEM, symbol template-rescue:R_200-formula
- removed U1: MCP2561-E_SN, footprints:SOIC-8_3.9x4.9mm_Pitch1.27mm_OEM, symbol template-rescue:MCP2561-E_SN-formula
- added D? (x2): BAS40-00, Package_TO_SOT_SMD:SOT-23, symbol formula:BAS40-00
- added U?: NanoFit_VT_TH_10, footprints:NanoFit_VT_10, symbol formula:NanoFit_VT_TH_10
Connections:
- net labels added: 3.3V, SS_HITL, VCCUSB
- net labels removed: CAN_HI, CAN_LO, CAN_RX, CAN_TX, SS_Accumulator, SS_Cockpit, SS_LVBox, SS_Sensing
- wire segments 95 -> 83
- no-connect marks 17 -> 16
Other:
- note added: "USB CONVERTER"
- note removed: "CAN TRANSCEIVER\n"
- note removed: "CONVERTER"
- note removed: "Do not populate"
- moved on the sheet: J1
