File: hardware_in_the_loop/boards/hitl_system_interface/oem_HitLInterface_board/HitLSystemInterfaceSchematic/SystemHitLInterface.sch (KiCad schematic (older format))
At the start: 47 parts, among them J1 CONN_02X03, J2 Conn_01x04_Female, J3 Conn_01x04_Female, J4 Barrel_Jack, J5 Conn_01x04_Female, U1 ATmega328P-AU, U101 TPS560430YF, U3 USB_MicroB, U4 FT232RL, U6 NanoFit_RA_TH_12, Y1 Crystal_SMD

Commit message: PCB Layout V2
Parts:
- U3: footprint Connectors_USB:USB_Micro-B_Molex-105017-0001 -> Connector_USB:USB_Micro-B_Molex-105133-0031
Changed lines of the file:
@@
 F 0 "U3" H 2207 7017 50  0000 C CNN
 F 1 "USB_MicroB" H 2207 6926 50  0000 C CNN
-F 2 "Connectors_USB:USB_Micro-B_Molex-105017-0001" H 2100 6900 50  0001 C CNN
+F 2 "Connector_USB:USB_Micro-B_Molex-105133-0031" H 2100 6900 50  0001 C CNN
 F 3 "https://www.molex.com/pdm_docs/sd/1050170001_sd.pdf" H 2100 6900 50  0001 C CNN
 F 4 "DK" H 2400 6300 50  0001 C CNN "MFN"
