File: hardware_in_the_loop/boards/hitl_system_interface/oem_HitLInterface_board/HitLSystemInterfaceSchematic/SystemHitLInterface.kicad_pcb (KiCad board)
At the start: 2 copper layers, 109.3 x 58.3 mm, 48 parts, among them J1 CONN_02X03, J2 Conn_01x04_Female, J3 Conn_01x04_Female, J4 Barrel_Jack, J5 Conn_01x04_Female, U1 ATmega328P-AU, U101 TPS560430YF, U3 USB_MicroB, U4 FT232RL, U6 NanoFit_RA_TH_12, Y1 Crystal_SMD

Commit message: HitL System PCB Layout Rev4 3-13-2021
Routing:
- net /SCK: track 102.6 -> 76.0 mm
- net Net-(F1-Pad1): track 28.7 -> 15.8 mm
- net /MOSI: track 66.3 -> 53.6 mm
- net VCC: track 182.5 -> 170.2 mm, vias 12 -> 7
- net /RESET: track 59.9 -> 51.6 mm
- net Net-(D1-Pad1): track 14.2 -> 7.24 mm
- net /D4: track 64.4 -> 59.7 mm
- net /MISO: track 67.9 -> 63.3 mm
- net /SDA: track 104.0 -> 99.7 mm
- net /D3: track 50.2 -> 46.3 mm
- net /RXD: track 36.3 -> 32.7 mm
- net /TXD: track 33.8 -> 30.5 mm
- net /AI3: track 35.1 -> 32.2 mm
- net /AI4: track 34.3 -> 31.4 mm
- net Net-(R4-Pad2): track 22.6 -> 19.9 mm
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