File: telemetry/can_replicator/can_replicator.kicad_pcb (KiCad board)
At the start: 2 copper layers, 109.3 x 58.3 mm, 19 parts, among them U101 TPS560430YF

Commit message: feat: begin layoutof components
Parts:
- removed C101, C103: C_0.1uF, footprints:C_0805_OEM
- removed C102: C_2.2uF, footprints:C_0603_1608Metric
- removed COUT101: C_22uF, footprints:C_1206_OEM
- removed COUT102: C_33uF, footprints:Fuse_1812
- removed COUT103: C_47uF, footprints:C_0805_OEM
- removed D101: D_Zener_18V, footprints:DO-214AA
- removed D102, D103: LED_0805, footprints:LED_0805_OEM
- removed F101: F_500mA_16V, footprints:Fuse_1210
- removed G***: LOGO, footprints:Logo_Large
- removed G***: LOGO, footprints:phoenix
- removed L101: L_100uH, footprints:L_100uH_OEM
- removed R101: R_1K, footprints:R_0805_OEM
- removed R102: R_25K, footprints:R_0805_OEM
- removed R103: R_100K, footprints:R_0805_OEM
- removed R104: R_0_2512, footprints:R_2512_OEM
- removed R105: R_200, footprints:R_0805_OEM
- removed U101: TPS560430YF, footprints:SOT-23-6_OEM
- added C1: C_0.1uF, footprints:C_0805_OEM, F.Cu at (85.0, 95.0)
- added C2: C_0.1uF, footprints:C_0805_OEM, F.Cu at (91.0, 79.0)
- added C3: C_100pF, footprints:C_0805_OEM, F.Cu at (94.0, 83.0)
- added C4: C_30pF, footprints:C_0805_OEM, F.Cu at (97.0, 127.0)
- added C5: C_30pF, footprints:C_0805_OEM, F.Cu at (99.0, 119.0)
- added C6: C_10nF, footprints:C_0805_OEM, F.Cu at (102.0, 71.0)
- added C7: C_100nF, footprints:C_0603_1608Metric, F.Cu at (131.0, 47.0)
- added C8: C_4.7uF, footprints:C_0603_1608Metric, F.Cu at (131.3, 49.9)
- added C9: C_100nF, footprints:C_0603_1608Metric, F.Cu at (148.0, 67.0)
- added D1: LED_0805_Amber, footprints:LED_0805_OEM, F.Cu at (152.1, 64.0)
- added D2: LED_0805_Amber, footprints:LED_0805_OEM, F.Cu at (152.1, 62.0)
- added D3: LED_0805, footprints:LED_0805_OEM, F.Cu at (96.0, 66.0)
- added D4: LED_0805, footprints:LED_0805_OEM, F.Cu at (119.0, 109.0)
- added D5: LED_0805, footprints:LED_0805_OEM, F.Cu at (119.0, 111.0)
- added D6: LED_0805, footprints:LED_0805_OEM, F.Cu at (119.0, 113.0)
- added J1: CONN_02X03, footprints:Pin_Header_Straight_2x03, F.Cu at (124.0, 95.0)
- added J2: MM_M_VT_20, footprints:micromatch_female_vert_20, F.Cu at (74.5, 88.0)
- added R1: R_100, footprints:R_0805_OEM, F.Cu at (90.0, 83.0)
- added R2: R_120_DNP, footprints:R_0805_OEM, F.Cu at (97.0, 95.0)
- added R3: R_10K, footprints:R_0805_OEM, F.Cu at (102.0, 78.0)
- added R4: R_200, footprints:R_0805_OEM, F.Cu at (125.0, 109.0)
- added R5: R_200, footprints:R_0805_OEM, F.Cu at (125.0, 111.0)
- added R6: R_200, footprints:R_0805_OEM, F.Cu at (125.0, 113.0)
- added R7: R_200, footprints:R_0805_OEM, F.Cu at (148.0, 64.0)
- added R8: R_200, footprints:R_0805_OEM, F.Cu at (148.0, 62.0)
- added R9: R_200, footprints:R_0805_OEM, F.Cu at (96.0, 70.0)
- added TP1: TP, footprints:tp_1.6mm, F.Cu at (109.0, 66.0)
- added TP2: TP, footprints:tp_1.6mm, F.Cu at (113.0, 66.0)
- added U1: MCP2561-E_SN, footprints:SOIC-8_3.9x4.9mm_Pitch1.27mm_OEM, F.Cu at (91.2, 94.8)
- added U2: ATMEGA16M1, footprints:TQFP-32_7x7mm_Pitch0.8mm, F.Cu at (103.3, 85.3)
- added U3: USB_MicroB, Connector_USB:USB_Micro-B_Molex-105017-0001, F.Cu at (102.0, 66.0)
- added U4: FT232RL, Package_SO:SSOP-28_5.3x10.2mm_P0.65mm, F.Cu at (140.0, 64.0)
- added Y1: Crystal_SMD, footprints:Crystal_SMD_FA238, F.Cu at (97.9, 123.2)
Routing:
- net GND: track 65.5 -> 25.5 mm, vias 11 -> 0
- net Net-(C101-Pad1): track 22.9 -> 0.00 mm
- net VCC: track 22.7 -> 0.00 mm
- net Net-(COUT101-Pad1): track 17.3 -> 0.00 mm
- net /12V: track 13.1 -> 0.00 mm
- net Net-(C103-Pad2): track 5.44 -> 0.00 mm
- net Net-(R102-Pad1): track 4.18 -> 0.00 mm
- net Net-(C103-Pad1): track 2.39 -> 0.00 mm
- net Net-(D103-Pad2): track 1.75 -> 0.00 mm
- net Net-(D102-Pad2): track 1.75 -> 0.00 mm
- removed copper zone on F.Cu, net GND
- removed copper zone on F.Cu, net Net-(C103-Pad1)
- removed copper zone on F.Cu, net Net-(C103-Pad2)
- removed copper zone on F.Cu, net Net-(COUT101-Pad1)
Other:
- board outline removed
- board text added: "1"
- board text added: "2"
- board text added: "3"
- board text added: "DEBUG"
- board text removed: "12V"
- board text removed: "5V"
- board text removed: "GND"
