File: telemetry/can_replicator/can_replicator.kicad_pcb (KiCad board)
At the start: 2 copper layers, 28.2 x 53.2 mm, 42 parts, among them J1 CONN_02X03, J2 MM_M_VT_20, J3 CONN_01X03, J4 CONN_01X03, U1 MCP2561-E_SN, U2 ATMEGA16M1, U3 USB_MicroB, U4 FT232RL, Y1 Crystal_SMD

Commit message: Small tweaks for fabbing
Parts:
- moved C7 14.9 mm to (100.6, 85.9), turned to 270 degrees
- moved C8 12.7 mm to (102.2, 85.9)
- moved R2 1.53 mm to (97.5, 96.1)
- moved C1 0.06 mm to (96.2, 115.0)
Routing:
- net /USBD-: track 21.9 -> 15.0 mm
- net +5V: track 153.8 -> 147.1 mm
- net /USBD+: track 20.9 -> 15.0 mm
- net /CAN_+: track 20.5 -> 19.9 mm
- net GND: track 52.4 -> 51.7 mm
- net /CAN_RX: track 9.12 -> 9.66 mm
