File: hardware_in_the_loop/boards_v2/primary_board/primary_board.sch (KiCad schematic (older format))
At the start: 22 parts

Commit message: Added all connectors and most components
Parts:
- removed C?: C_0.1uF, footprints:C_0805_OEM, symbol formula:C_0.1uF
- removed J?: CONN_01X03, Pin_Headers:Pin_Header_Straight_1x03_Pitch2.54mm, symbol formula:CONN_01X03
- removed J?: SSW-120-01-F-D, footprints:SAMTEC_SSW-120-01-F-D, symbol formula:SSW-120-01-F-D
- removed U?: LTC2489CDEPBF, footprints:DFN-14_DE_AD, symbol formula:LTC2489CDEPBF
- removed U?: 74HCT4051, footprints:TSSOP-16-OEM, symbol formula:74HCT4051
- added C11, C12: C_30pF, footprints:C_0805_OEM, symbol formula:C_30pF
- added C13: C_0.1uF, footprints:C_0805_OEM, symbol formula:C_0.1uF
- added C14, C16: C_10uF_25V, footprints:C_0805_OEM, symbol formula:C_10uF_25V
- added C15: C_4.7uF_25V, footprints:C_0805_OEM, symbol formula:C_4.7uF_25V
- added C3, C4: C_10uF_50V, footprints:C_0805_OEM, symbol formula:C_10uF_50V
- added D1, D2: LED_0805, footprints:LED_0805_OEM, symbol formula:LED_0805
- added D3: LED_0805_Red, footprints:LED_0805_OEM, symbol formula:LED_0805_Red
- added D4, D5: LED_0805_Amber, footprints:LED_0805_OEM, symbol formula:LED_0805_Amber
- added F1: 1.5A_Fuse, footprints:Fuse_1206, symbol formula:1.5A_Fuse
- added J2: Barrel_jack, footprints:barrel_jack_PJ-037A, symbol formula:Barrel_jack
- added J3, J4, J5, J6, J7: CONN_01X03, footprints:PinHeader_1x03_P2.54mm_Vertical, symbol formula:CONN_01X03
- added J8: DSub-9, footprints:TE_5745781-4, symbol formula:DSub-9
- added J9: SSW-122-01-G-D, footprints:SAMTEC_SSW-122-01-G-D, symbol formula:SSW-122-01-G-D
- added Q1, Q2, Q3, Q4: SSM3K333R, footprints:SOT-23F, symbol formula:SSM3K333R
- added R10, R13, R15: R_12K, footprints:R_0805_OEM, symbol formula:R_12K
- added R11, R16: R_3.01K, footprints:R_0805_OEM, symbol formula:R_3.01K
- added R12: R_1M, footprints:R_0805_OEM, symbol formula:R_1M
- added R14, R20, R22, R7: R_1.91K, footprints:R_0805_OEM, symbol formula:R_1.91K
- added R17: R_120_DNP, footprints:R_0805_OEM, symbol formula:R_120_DNP
- added R18: R_39K, footprints:R_0805_OEM, symbol formula:R_39K
- added R19, R21, R4, R6, R8: R_10K, footprints:R_0805_OEM, symbol formula:R_10K
- added U3: LT3045, footprints:MSOP-12_MSE, symbol formula:LT3045
- added Y1: Crystal_12MHz, footprints:Crystal_SMD_FA238, symbol formula:Crystal_12MHz
- gave numbers to parts that had none: 17
Connections:
- net +5V: now also U1.30 (VBUS-DET), J7.3 (P3), R10.2; no longer U2.3 (VDD), U2.4 (VLOGIC), U4.36 (V+)
- net ADC1: now also J9.36
- net ADC2: now also J9.35
- net Analog-MUX1: now also J9.38
- net Analog-MUX2: now also J9.37
- net Analog-MUX3: now also J9.40
- net Analog-MUX4: now also J9.39
- net GND: now also R3.1, R5.1, U2.13 (GND), U2.14 (RSTSL), U2.8 (GAIN), C11.2, C12.2, C13.2, C14.2, C15.2, C16.2, C3.2, C4.2, D2.1 (K), J2.2 (Shell), J3.3 (P3), J4.3 (P3), J5.3 (P3), J6.3 (P3), J8.3, J8.6, J9.01, J9.02, J9.25, J9.26, J9.41, Q1.2 (S), Q2.2 (S), Q3.2 (S), Q4.2 (S), R11.2, R13.2, R16.2, R18.2, R19.2, R21.2, R4.2, R6.2, U3.13 (GND), U3.6 (ILIM), U3.9 (GND), Y1.2, Y1.4
- net GPIO-1: now also J9.03
- net GPIO-10: now also J9.12
- net GPIO-11: now also J9.13
- net GPIO-12: now also J9.14
- net GPIO-13: now also J9.15
- net GPIO-14: now also J9.16
- net GPIO-15: now also J9.17
- net GPIO-16: now also J9.18
- net GPIO-17: now also J9.19
- net GPIO-18: now also J9.20
- net GPIO-19: now also J9.21
- net GPIO-2: now also J9.04
- net GPIO-20: now also J9.22
- net GPIO-21: now also J9.23
- net GPIO-22: now also J9.24
- net GPIO-25: now also Q3.1 (G), R19.1
- net GPIO-27: now also Q4.1 (G), R21.1
- net GPIO-3: now also J9.05
- net GPIO-4: now also J9.06
- net GPIO-5: now also J9.07
- net GPIO-6: now also J9.08
- net GPIO-7: now also J9.09
- net GPIO-8: now also J9.10
- net GPIO-9: now also J9.11
- net VOUT-1: now also J9.27
- net VOUT-2: now also J9.28
- net VOUT-3: now also J9.29
- net VOUT-4: now also J9.30
- net VOUT-5: now also J9.31
- net VOUT-6: now also J9.32
- net VOUT-7: now also J9.33
- net VOUT-8: now also J9.34
- net FT-GPIO2: now reaches U1.15 (GPIO2/SS3O/SUSP-OUT)
- net FT-GPIO2: now also Q2.1 (G), R6.1
- net FT-GPIO3: now reaches U1.16 (GPIO3/WAKEUP/INTR)
- net FT-GPIO3: now also Q1.1 (G), R4.1
- net at U1.18 (XSCI): now also C12.1, R12.1, Y1.3
- net at U1.19 (XSCO): now also C11.1, R12.2, Y1.1
- net at U1.21 (RREF): now also R13.1
- net FT-VPP: now reaches U1.29 (VPP)
- net DAC-LDAC: now reaches U2.15 (LDAC_n)
- net DAC-LDAC: now also Q2.3 (D), R8.2
- net VBUS: now reaches U2.17 (RESET_n)
- net VBUS: now also U2.18 (VREF), U2.3 (VDD), U2.4 (VLOGIC), U4.36 (V+), C13.1, C14.1, C16.1, J3.1 (P1), J4.1 (P1), J5.1 (P1), J6.1 (P1), R8.1, U3.10 (OUTS), U3.11 (OUT), U3.12 (OUT)
- net DAC-A0: now reaches U2.6 (A0)
- net DAC-A0: now also J3.2 (P2)
- net DAC-A1: now reaches U2.7 (A1)
- net DAC-A1: now also J4.2 (P2)
- net at U4.1 (ISET): now also R18.1
- net GPIO-AD1: now reaches U4.35 (AD1)
- net GPIO-AD1: now also J6.2 (P2)
- net GPIO-AD0: now reaches U4.4 (AD0)
- net GPIO-AD0: now also J5.2 (P2)
- new net: D3.1 (K), Q1.3 (D)
- new net: D3.2 (A), R7.2
- new net: F1.1, J2.1 (center)
- new net: D4.1 (K), Q3.3 (D)
- new net: D4.2 (A), R20.2
- new net: D5.1 (K), Q4.3 (D)
- new net: D5.2 (A), R22.2
- new net: D2.2 (A), R14.2
- new net +12V: C3.1, C4.1, F1.2, J7.1 (P1), J9.42, R14.1, R15.1, R20.1, R22.1, R7.1
- new net Analog-MUX5: R15.2, R16.1
- new net Analog-MUX6: R10.1, R11.1
- new net CANH+: J8.7, J9.43, R17.1
- new net CANL-: J8.2, J9.44, R17.2
- new net Lin-IN: C15.1, J7.2 (P2), U3.1 (IN), U3.2 (IN), U3.3 (IN), U3.4 (EN/UV), U3.7 (PGFB)
- no-connect marks 11 -> 14
Other:
- note added: "5V (output)"
- note added: "Gain = 1"
- note added: "I2C packages pin capacitance?"
- note added: "Operating in Mode 0\nSee pg.13 for more info"
- note added: "Output protection?"
- note added: "Parts to add:\n- I2C Level Shifter\n- 33.2K res\n- 49.9K res"
- note added: "Should we add more address options?\nThere are currently 4 which would cover\nthe entire vehicle"
- note added: "Sink 10mA\nSource 4.5mA"
- note added: "Vout = Vin * ~~0.2\nVout ≈ 1V"
- note added: "Vout = Vin * ~~0.2\nVout ≈ 2.4V"
- note added: "Vout0 thru Vout3 can Source/Sink 40mA\nVout4 thru Vout7 can Source/Sink 40mA"
- note added: "https://www.digikey.com/en/products/detail/samtec-inc/SSW-122-01-G-D/1112036\n"
- note added: "https://www.digikey.com/en/products/detail/w%C3%BCrth-elektronik/61304421121/4846887"
- note added: "~~5mA"
- note removed: "Add voltage divider for ADC\n"
- note removed: "Parts to add:\n- 12MHz Crystal\n- 3.3V/5V Lin\n- I2C Level Shifter"
- moved on the sheet: C10, C5, C6, C7, C8, C9, R9, U2, U4
